File: z80.sch (KiCad schematic (older format))
At the start: 24 parts, among them J5 USB_B, J6 PWR, SW1 KS01Q, U1 Z80CPU, U16 74AHC08, U2 74AHC14, U3 SST39SF010, U4 74AHC32, U5 AS6C1008-55PCN, U6 74AHC138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

Commit message: Latest rev of z80 schematic.
git-svn-id: svn+ssh://dev.thehead.ca/depot/main/z80@613 995eaefb-0ce2-40e3-b8bc-69bf8729875b
Parts:
- removed U16: 74AHC08, symbol 74LS08
- added unit 3 of U4
Connections:
- net A13: now also U4.9
- net A14: now also U4.10; no longer U4.1
- net GND: now also U4.7 (GND)
- net VCC: now also U4.14 (VCC)
- new net: U4.1, U4.8
- no-connect marks 15 -> 12
Changed lines of the file:
@@
 $Descr USLetter 11000 8500
 encoding utf-8
-Sheet 1 6
+Sheet 1 7
 Title "Z80 Prototype"
-Date "2017-10-22"
-Rev "4"
+Date "2017-10-24"
+Rev "5"
 Comp ""
 Comment1 ""
@@
 	1    0    0    -1
 $EndComp
-$Comp
-L GND #PWR09
-U 1 1 59B5E817
-P 600 7750
-F 0 "#PWR09" H 600 7500 50  0001 C CNN
-F 1 "GND" H 600 7600 50  0000 C CNN
-F 2 "" H 600 7750 50  0001 C CNN
-F 3 "" H 600 7750 50  0001 C CNN
-	1    600  7750
-	1    0    0    -1
-$EndComp
 NoConn ~ 3050 3950
 $Comp
-L VCC #PWR010
+L VCC #PWR09
 U 1 1 59B5EB83
 P 2950 3850
-F 0 "#PWR010" H 2950 3700 50  0001 C CNN
+F 0 "#PWR09" H 2950 3700 50  0001 C CNN
 F 1 "VCC" H 2950 4000 50  0000 C CNN
 F 2 "" H 2950 3850 50  0001 C CNN
@@
 NoConn ~ 3050 2650
 $Comp
-L VCC #PWR011
+L VCC #PWR010
 U 1 1 59B5EC49
 P 2950 2750
-F 0 "#PWR011" H 2950 2600 50  0001 C CNN
+F 0 "#PWR010" H 2950 2600 50  0001 C CNN
 F 1 "VCC" H 2950 2900 50  0000 C CNN
 F 2 "" H 2950 2750 50  0001 C CNN
@@
 $EndComp
 $Comp
-L VCC #PWR012
+L VCC #PWR011
 U 1 1 59B5ECC3
 P 2950 2150
-F 0 "#PWR012" H 2950 2000 50  0001 C CNN
+F 0 "#PWR011" H 2950 2000 50  0001 C CNN
 F 1 "VCC" H 2950 2300 50  0000 C CNN
 F 2 "" H 2950 2150 50  0001 C CNN
@@
 NoConn ~ 5400 3250
 $Comp
-L GND #PWR013
+L GND #PWR012
 U 1 1 59B6D08B
 P 5250 3150
-F 0 "#PWR013" H 5250 2900 50  0001 C CNN
+F 0 "#PWR012" H 5250 2900 50  0001 C CNN
 F 1 "GND" H 5250 3000 50  0000 C CNN
 F 2 "" H 5250 3150 50  0001 C CNN
@@
 A13
 $Comp
-L VCC #PWR014
+L VCC #PWR013
 U 1 1 59B7E032
 P 5250 3550
-F 0 "#PWR014" H 5250 3400 50  0001 C CNN
+F 0 "#PWR013" H 5250 3400 50  0001 C CNN
 F 1 "VCC" H 5250 3700 50  0000 C CNN
 F 2 "" H 5250 3550 50  0001 C CNN
@@
 	-1   0    0    -1
 $EndComp
-Text Label 8400 850  2    60   ~ 0
-A14
+Text Label 9600 750  2    60   ~ 0
+A13
 $Comp
 L AS6C1008-55SIN U5
@@
 $EndComp
 $Comp
-L GND #PWR015
+L GND #PWR014
 U 1 1 59B81476
 P 8700 3150
-F 0 "#PWR015" H 8700 2900 50  0001 C CNN
+F 0 "#PWR014" H 8700 2900 50  0001 C CNN
 F 1 "GND" H 8700 3000 50  0000 C CNN
 F 2 "" H 8700 3150 50  0001 C CNN
@@
 $EndComp
 $Comp
-L VCC #PWR016
+L VCC #PWR015
 U 1 1 59B81557
 P 8700 3050
-F 0 "#PWR016" H 8700 2900 50  0001 C CNN
+F 0 "#PWR015" H 8700 2900 50  0001 C CNN
 F 1 "VCC" H 8700 3200 50  0000 C CNN
 F 2 "" H 8700 3050 50  0001 C CNN
@@
 $EndComp
 $Comp
-L GND #PWR017
+L GND #PWR016
 U 1 1 59B816F6
 P 7400 3150
-F 0 "#PWR017" H 7400 2900 50  0001 C CNN
+F 0 "#PWR016" H 7400 2900 50  0001 C CNN
 F 1 "GND" H 7400 3000 50  0000 C CNN
 F 2 "" H 7400 3150 50  0001 C CNN
@@
 Connection ~ 3250 7800
 Wire Wire Line
-	8250 850  8400 850
+	9450 750  9600 750
 Wire Wire Line
 	5000 3750 5400 3750
@@
 $EndComp
 $Comp
-L GND #PWR018
+L GND #PWR017
 U 1 1 59CD39B1
 P 1350 4450
-F 0 "#PWR018" H 1350 4200 50  0001 C CNN
+F 0 "#PWR017" H 1350 4200 50  0001 C CNN
 F 1 "GND" H 1350 4300 50  0000 C CNN
 F 2 "" H 1350 4450 50  0001 C CNN
@@
 $EndComp
 $Comp
-L VCC #PWR019
+L VCC #PWR018
 U 1 1 59CD3A52
 P 1350 3850
-F 0 "#PWR019" H 1350 3700 50  0001 C CNN
+F 0 "#PWR018" H 1350 3700 50  0001 C CNN
 F 1 "VCC" H 1350 4000 50  0000 C CNN
 F 2 "" H 1350 3850 50  0001 C CNN
@@
 	2950 5650 2850 5650
 $Comp
-L VCC #PWR020
+L VCC #PWR019
 U 1 1 59D3FEB7
 P 2800 5550
-F 0 "#PWR020" H 2800 5400 50  0001 C CNN
+F 0 "#PWR019" H 2800 5400 50  0001 C CNN
 F 1 "VCC" H 2800 5700 50  0000 C CNN
 F 2 "" H 2800 5550 50  0001 C CNN
@@
 CLK
 $Comp
-L VCC #PWR021
+L VCC #PWR020
 U 1 1 59D7BD8F
 P 7800 5000
-F 0 "#PWR021" H 7800 4850 50  0001 C CNN
+F 0 "#PWR020" H 7800 4850 50  0001 C CNN
 F 1 "VCC" H 7800 5150 50  0000 C CNN
 F 2 "" H 7800 5000 50  0001 C CNN
@@
 	3050 2250 2750 2250
 $Comp
-L VCC #PWR022
+L VCC #PWR021
 U 1 1 59D85B4D
 P 2450 2250
-F 0 "#PWR022" H 2450 2100 50  0001 C CNN
+F 0 "#PWR021" H 2450 2100 50  0001 C CNN
 F 1 "VCC" H 2450 2400 50  0000 C CNN
 F 2 "" H 2450 2250 50  0001 C CNN
@@
 	1    0    0    -1
 $EndComp
-$Comp
-L 74LS08 U16
-U 2 1 59D86740
-P 1200 6350
-F 0 "U16" H 1200 6400 50  0000 C CNN
-F 1 "74AHC08" H 1200 6300 50  0000 C CNN
-F 2 "" H 1200 6350 50  0001 C CNN
-F 3 "" H 1200 6350 50  0001 C CNN
-	2    1200 6350
-	1    0    0    -1
-$EndComp
-$Comp
-L 74LS08 U16
-U 3 1 59D86924
-P 1200 6800
-F 0 "U16" H 1200 6850 50  0000 C CNN
-F 1 "74AHC08" H 1200 6750 50  0000 C CNN
-F 2 "" H 1200 6800 50  0001 C CNN
-F 3 "" H 1200 6800 50  0001 C CNN
-	3    1200 6800
-	1    0    0    -1
-$EndComp
-$Comp
-L 74LS08 U16
-U 4 1 59D8692A
-P 1200 7300
-F 0 "U16" H 1200 7350 50  0000 C CNN
-F 1 "74AHC08" H 1200 7250 50  0000 C CNN
-F 2 "" H 1200 7300 50  0001 C CNN
-F 3 "" H 1200 7300 50  0001 C CNN
-	4    1200 7300
-	1    0    0    -1
-$EndComp
-NoConn ~ 1800 7300
-NoConn ~ 1800 6800
-NoConn ~ 1800 6350
-Connection ~ 600  6900
 $Comp
 L C C26
@@
 Wire Bus Line
 	9250 4300 9150 4300
-Wire Wire Line
-	600  6250 600  7750
-Connection ~ 600  6450
-Connection ~ 600  6700
-Connection ~ 600  7400
-Connection ~ 600  7200
 $Comp
 L USB_B J5
@@
 	1    0    0    -1
 $EndComp
+$Sheet
+S 600  7650 550  250
+U 59EFC926
+F0 "Spares" 60
+F1 "spares.sch" 60
+$EndSheet
+$Comp
+L 74LS32 U4
+U 3 1 59EFDDD2
+P 8850 850
+F 0 "U4" H 8850 900 50  0000 C CNN
+F 1 "74AHC32" H 8850 800 50  0000 C CNN
+F 2 "" H 8850 850 50  0001 C CNN
+F 3 "" H 8850 850 50  0001 C CNN
+	3    8850 850
+	-1   0    0    -1
+$EndComp
+Text Label 9600 950  2    60   ~ 0
+A14
+Wire Wire Line
+	9450 950  9600 950
 $EndSCHEMATC

Commit message: Add expansion bus connector; rev 6.
git-svn-id: svn+ssh://dev.thehead.ca/depot/main/z80@616 995eaefb-0ce2-40e3-b8bc-69bf8729875b
Parts:
- added J3: Conn_02x20_Top_Bottom, symbol Conn_02x20_Top_Bottom
Connections:
- net A0: now also J3.2 (Pin_2)
- net A1: now also J3.3 (Pin_3)
- net A10: now also J3.12 (Pin_12)
- net A11: now also J3.13 (Pin_13)
- net A12: now also J3.14 (Pin_14)
- net A13: now also J3.15 (Pin_15)
- net A14: now also J3.16 (Pin_16)
- net A15: now also J3.17 (Pin_17)
- net A2: now also J3.4 (Pin_4)
- net A3: now also J3.5 (Pin_5)
- net A4: now also J3.6 (Pin_6)
- net A5: now also J3.7 (Pin_7)
- net A6: now also J3.8 (Pin_8)
- net A7: now also J3.9 (Pin_9)
- net A8: now also J3.10 (Pin_10)
- net A9: now also J3.11 (Pin_11)
- net CLK: now also J3.39 (Pin_39)
- net D0: now also J3.21 (Pin_21)
- net D1: now also J3.22 (Pin_22)
- net D2: now also J3.23 (Pin_23)
- net D3: now also J3.24 (Pin_24)
- net D4: now also J3.25 (Pin_25)
- net D5: now also J3.26 (Pin_26)
- net D6: now also J3.27 (Pin_27)
- net D7: now also J3.28 (Pin_28)
- net GND: now also J3.40 (Pin_40)
- net VCC: now also J3.1 (Pin_1)
- net ~INT: now also J3.20 (Pin_20)
- net ~IORQ: now also J3.32 (Pin_32)
- net ~M1: now also J3.38 (Pin_38)
- net ~MREQ: now also J3.31 (Pin_31)
- net ~RD: now also J3.29 (Pin_29)
- net ~RESET: now also J3.19 (Pin_19)
- net ~WR: now also J3.30 (Pin_30)
- no-connect marks 12 -> 18
Changed lines of the file:
@@
 Sheet 1 7
 Title "Z80 Prototype"
-Date "2017-10-24"
-Rev "5"
+Date "2018-03-28"
+Rev "6"
 Comp ""
 Comment1 ""
@@
 Wire Wire Line
 	9450 950  9600 950
+$Comp
+L Conn_02x20_Top_Bottom J3
+U 1 1 5ABBD7C9
+P 9750 2450
+F 0 "J3" H 9800 3450 50  0000 C CNN
+F 1 "Conn_02x20_Top_Bottom" H 9800 1350 50  0000 C CNN
+F 2 "" H 9750 2450 50  0001 C CNN
+F 3 "" H 9750 2450 50  0001 C CNN
+	1    9750 2450
+	1    0    0    -1
+$EndComp
+Wire Wire Line
+	9550 1550 9300 1550
+Wire Wire Line
+	9550 1650 9300 1650
+Wire Wire Line
+	9550 1750 9300 1750
+Wire Wire Line
+	9550 1850 9300 1850
+Wire Wire Line
+	9550 1950 9300 1950
+Wire Wire Line
+	9550 2050 9300 2050
+Wire Wire Line
+	9550 2150 9300 2150
+Wire Wire Line
+	9550 2250 9300 2250
+Wire Wire Line
+	9550 2350 9300 2350
+Wire Wire Line
+	9550 2450 9300 2450
+Wire Wire Line
+	9550 2550 9300 2550
+Wire Wire Line
+	9550 2650 9300 2650
+Wire Wire Line
+	9550 2750 9300 2750
+Wire Wire Line
+	9550 2850 9300 2850
+Wire Wire Line
+	9550 2950 9300 2950
+Wire Wire Line
+	9550 3050 9300 3050
+Wire Wire Line
+	9550 3150 9300 3150
+Wire Wire Line
+	9550 3250 9300 3250
+Wire Wire Line
+	9550 3350 9300 3350
+Wire Wire Line
+	9550 3450 9300 3450
+Wire Wire Line
+	10050 1550 10300 1550
+Wire Wire Line
+	10050 1650 10300 1650
+Wire Wire Line
+	10050 1750 10300 1750
+Wire Wire Line
+	10050 1850 10300 1850
+Wire Wire Line
+	10050 1950 10300 1950
+Wire Wire Line
+	10050 2050 10300 2050
+Wire Wire Line
+	10050 2150 10300 2150
+Wire Wire Line
+	10050 2250 10300 2250
+Wire Wire Line
+	10050 2350 10300 2350
+Wire Wire Line
+	10050 2450 10300 2450
+Wire Wire Line
+	10050 2550 10300 2550
+Wire Wire Line
+	10050 2650 10300 2650
+Wire Wire Line
+	10050 2750 10300 2750
+Wire Wire Line
+	10050 2850 10300 2850
+Wire Wire Line
+	10050 2950 10300 2950
+Wire Wire Line
+	10050 3050 10300 3050
+Wire Wire Line
+	10050 3150 10300 3150
+Wire Wire Line
+	10050 3250 10300 3250
+Wire Wire Line
+	10050 3350 10300 3350
+Wire Wire Line
+	10050 3450 10300 3450
+$Comp
+L VCC #PWR022
+U 1 1 5ABBE8C3
+P 9300 1550
+F 0 "#PWR022" H 9300 1400 50  0001 C CNN
+F 1 "VCC" H 9300 1700 50  0000 C CNN
+F 2 "" H 9300 1550 50  0001 C CNN
+F 3 "" H 9300 1550 50  0001 C CNN
+	1    9300 1550
+	1    0    0    -1
+$EndComp
+$Comp
+L GND #PWR023
+U 1 1 5ABBEB83
+P 10300 3450
+F 0 "#PWR023" H 10300 3200 50  0001 C CNN
+F 1 "GND" H 10300 3300 50  0000 C CNN
+F 2 "" H 10300 3450 50  0001 C CNN
+F 3 "" H 10300 3450 50  0001 C CNN
+	1    10300 3450
+	1    0    0    -1
+$EndComp
+Text Label 9300 1650 0    60   ~ 0
+A0
+Text Label 9300 1750 0    60   ~ 0
+A1
+Text Label 9300 1850 0    60   ~ 0
+A2
+Text Label 9300 1950 0    60   ~ 0
+A3
+Text Label 9300 2050 0    60   ~ 0
+A4
+Text Label 9300 2150 0    60   ~ 0
+A5
+Text Label 9300 2250 0    60   ~ 0
+A6
+Text Label 9300 2350 0    60   ~ 0
+A7
+Text Label 9300 2450 0    60   ~ 0
+A8
+Text Label 9300 2550 0    60   ~ 0
+A9
+Text Label 9300 2650 0    60   ~ 0
+A10
+Text Label 9300 2750 0    60   ~ 0
+A11
+Text Label 9300 2850 0    60   ~ 0
+A12
+Text Label 9300 2950 0    60   ~ 0
+A13
+Text Label 9300 3050 0    60   ~ 0
+A14
+Text Label 9300 3150 0    60   ~ 0
+A15
+Text Label 10300 1550 2    60   ~ 0
+D0
+Text Label 10300 1650 2    60   ~ 0
+D1
+Text Label 10300 1750 2    60   ~ 0
+D2
+Text Label 10300 1850 2    60   ~ 0
+D3
+Text Label 10300 1950 2    60   ~ 0
+D4
+Text Label 10300 2050 2    60   ~ 0
+D5
+Text Label 10300 2150 2    60   ~ 0
+D6
+Text Label 10300 2250 2    60   ~ 0
+D7
+Text Label 9300 3350 0    60   ~ 0
+~RESET
+Text Label 9300 3450 0    60   ~ 0
+~INT
+Text Label 10300 3350 2    60   ~ 0
+CLK
+Text Label 10300 3250 2    60   ~ 0
+~M1
+Text Label 10300 2350 2    60   ~ 0
+~RD
+Text Label 10300 2450 2    60   ~ 0
+~WR
+Text Label 10300 2550 2    60   ~ 0
+~MREQ
+Text Label 10300 2650 2    60   ~ 0
+~IORQ
+NoConn ~ 9300 3250
+NoConn ~ 10300 2750
+NoConn ~ 10300 2850
+NoConn ~ 10300 2950
+NoConn ~ 10300 3050
+NoConn ~ 10300 3150
 $EndSCHEMATC

Commit message: Assign footprints to schematic, drawing custom connector, socket, and switch footprints as needed.
git-svn-id: svn+ssh://dev.thehead.ca/depot/main/z80@617 995eaefb-0ce2-40e3-b8bc-69bf8729875b
Parts:
- removed J3: Conn_02x20_Top_Bottom, symbol Conn_02x20_Top_Bottom
- added J3: Conn_02x20_Odd_Even, Pin_Headers:Pin_Header_Straight_2x20_Pitch2.54mm, symbol Conn_02x20_Odd_Even
- C1, C2, C24, C26, C3, C4, C5, C6, C7: footprint (none) -> Capacitors_THT:C_Disc_D4.3mm_W1.9mm_P5.00mm
- D1: footprint (none) -> LEDs:LED_D5.0mm
- J5: footprint (none) -> z80_footprints:USB_B_E8144-B02022-L
- J6: footprint (none) -> Pin_Headers:Pin_Header_Straight_2x01_Pitch2.54mm
- R1, R18, R29: footprint (none) -> Resistors_THT:R_Axial_DIN0204_L3.6mm_D1.6mm_P5.08mm_Horizontal
- SW1: footprint (none) -> z80_footprints:KS-01Q-02
- U1: footprint (none) -> Housings_DIP:DIP-40_W15.24mm_Socket_LongPads
- U2, U4: footprint (none) -> Housings_DIP:DIP-14_W7.62mm_LongPads
- U3, U5: footprint (none) -> Housings_DIP:DIP-32_W15.24mm_Socket_LongPads
- U6: footprint (none) -> Housings_DIP:DIP-16_W7.62mm_LongPads
Connections:
- net A0: now also J3.3 (Pin_3)
- net A1: now also J3.5 (Pin_5)
- net A10: now also J3.23 (Pin_23)
- net A11: now also J3.25 (Pin_25)
- net A12: now also J3.27 (Pin_27)
- net A13: now also J3.29 (Pin_29)
- net A14: now also J3.31 (Pin_31)
- net A15: now also J3.33 (Pin_33)
- net A2: now also J3.7 (Pin_7)
- net A3: now also J3.9 (Pin_9)
- net A4: now also J3.11 (Pin_11)
- net A5: now also J3.13 (Pin_13)
- net A6: now also J3.15 (Pin_15)
- net A7: now also J3.17 (Pin_17)
- net A8: now also J3.19 (Pin_19)
- net A9: now also J3.21 (Pin_21)
- net CLK: now also J3.38 (Pin_38)
- net D0: now also J3.2 (Pin_2)
- net D1: now also J3.4 (Pin_4)
- net D2: now also J3.6 (Pin_6)
- net D3: now also J3.8 (Pin_8)
- net D4: now also J3.10 (Pin_10)
- net D5: now also J3.12 (Pin_12)
- net D6: now also J3.14 (Pin_14)
- net D7: now also J3.16 (Pin_16)
- net GND: now also J3.40 (Pin_40)
- net VCC: now also J3.1 (Pin_1)
- net ~INT: now also J3.39 (Pin_39)
- net ~IORQ: now also J3.24 (Pin_24)
- net ~M1: now also J3.36 (Pin_36)
- net ~MREQ: now also J3.22 (Pin_22)
- net ~RD: now also J3.18 (Pin_18)
- net ~RESET: now also J3.37 (Pin_37)
- net ~WR: now also J3.20 (Pin_20)
Changed lines of the file:
@@
 Sheet 1 7
 Title "Z80 Prototype"
-Date "2018-03-28"
-Rev "6"
+Date "2018-04-11"
+Rev "7"
 Comp ""
 Comment1 ""
@@
 F 0 "U1" H 3200 4150 50  0000 L CNN
 F 1 "Z80CPU" H 4000 4150 50  0000 L CNN
-F 2 "" H 3750 3150 50  0001 C CNN
+F 2 "Housings_DIP:DIP-40_W15.24mm_Socket_LongPads" H 3750 3150 50  0001 C CNN
 F 3 "" H 3750 3150 50  0001 C CNN
 	1    3750 2750
@@
 F 0 "SW1" H 850 1250 50  0000 L CNN
 F 1 "KS01Q" H 800 1090 50  0000 C CNN
-F 2 "" H 800 1350 50  0001 C CNN
+F 2 "z80_footprints:KS-01Q-02" H 800 1350 50  0001 C CNN
 F 3 "" H 800 1350 50  0001 C CNN
 	1    800  1150
@@
 F 0 "U2" H 1750 1250 50  0000 C CNN
 F 1 "74AHC14" H 1800 1050 50  0000 C CNN
-F 2 "" H 1600 1150 50  0001 C CNN
+F 2 "Housings_DIP:DIP-14_W7.62mm_LongPads" H 1600 1150 50  0001 C CNN
 F 3 "http://www.ti.com/lit/ds/symlink/sn74ahc14.pdf" H 1600 1150 50  0001 C CNN
 	1    1600 1150
@@
 F 0 "C1" H 1175 1550 50  0000 L CNN
 F 1 "0.1uF" H 1175 1350 50  0000 L CNN
-F 2 "" H 1188 1300 50  0001 C CNN
+F 2 "Capacitors_THT:C_Disc_D4.3mm_W1.9mm_P5.00mm" H 1188 1300 50  0001 C CNN
 F 3 "" H 1150 1450 50  0001 C CNN
 	1    1150 1450
@@
 F 0 "R1" V 1230 850 50  0000 C CNN
 F 1 "1M" V 1150 850 50  0000 C CNN
-F 2 "" V 1080 850 50  0001 C CNN
+F 2 "Resistors_THT:R_Axial_DIN0204_L3.6mm_D1.6mm_P5.08mm_Horizontal" V 1080 850 50  0001 C CNN
 F 3 "" H 1150 850 50  0001 C CNN
 	1    1150 850
@@
 F 0 "C2" H 2675 7750 50  0000 L CNN
 F 1 "0.1uF" H 2675 7550 50  0000 L CNN
-F 2 "" H 2688 7500 50  0001 C CNN
+F 2 "Capacitors_THT:C_Disc_D4.3mm_W1.9mm_P5.00mm" H 2688 7500 50  0001 C CNN
 F 3 "" H 2650 7650 50  0001 C CNN
 	1    2650 7650
@@
 F 0 "C3" H 2975 7750 50  0000 L CNN
 F 1 "0.1uF" H 2975 7550 50  0000 L CNN
-F 2 "" H 2988 7500 50  0001 C CNN
+F 2 "Capacitors_THT:C_Disc_D4.3mm_W1.9mm_P5.00mm" H 2988 7500 50  0001 C CNN
 F 3 "" H 2950 7650 50  0001 C CNN
 	1    2950 7650
@@
 F 0 "U2" H 2750 1250 50  0000 C CNN
 F 1 "74AHC14" H 2800 1050 50  0000 C CNN
-F 2 "" H 2600 1150 50  0001 C CNN
+F 2 "Housings_DIP:DIP-14_W7.62mm_LongPads" H 2600 1150 50  0001 C CNN
 F 3 "" H 2600 1150 50  0001 C CNN
 	2    2600 1150
@@
 F 0 "U3" H 6000 4050 50  0000 C CNN
 F 1 "SST39SF010" H 6000 1550 50  0000 C CNN
-F 2 "" H 6000 3050 50  0001 C CNN
+F 2 "Housings_DIP:DIP-32_W15.24mm_Socket_LongPads" H 6000 3050 50  0001 C CNN
 F 3 "" H 6000 3050 50  0001 C CNN
 	1    6000 2750
@@
 F 0 "C4" H 3275 7750 50  0000 L CNN
 F 1 "0.1uF" H 3275 7550 50  0000 L CNN
-F 2 "" H 3288 7500 50  0001 C CNN
+F 2 "Capacitors_THT:C_Disc_D4.3mm_W1.9mm_P5.00mm" H 3288 7500 50  0001 C CNN
 F 3 "" H 3250 7650 50  0001 C CNN
 	1    3250 7650
@@
 F 0 "U4" H 7650 1000 50  0000 C CNN
 F 1 "74AHC32" H 7650 900 50  0000 C CNN
-F 2 "" H 7650 950 50  0001 C CNN
+F 2 "Housings_DIP:DIP-14_W7.62mm_LongPads" H 7650 950 50  0001 C CNN
 F 3 "" H 7650 950 50  0001 C CNN
 	1    7650 950
@@
 F 0 "C5" H 3575 7750 50  0000 L CNN
 F 1 "0.1uF" H 3575 7550 50  0000 L CNN
-F 2 "" H 3588 7500 50  0001 C CNN
+F 2 "Capacitors_THT:C_Disc_D4.3mm_W1.9mm_P5.00mm" H 3588 7500 50  0001 C CNN
 F 3 "" H 3550 7650 50  0001 C CNN
 	1    3550 7650
@@
 F 0 "U4" H 6300 900 50  0000 C CNN
 F 1 "74AHC32" H 6300 800 50  0000 C CNN
-F 2 "" H 6300 850 50  0001 C CNN
+F 2 "Housings_DIP:DIP-14_W7.62mm_LongPads" H 6300 850 50  0001 C CNN
 F 3 "" H 6300 850 50  0001 C CNN
 	2    6300 850
@@
 F 0 "U5" H 8000 1489 50  0000 C BNN
 F 1 "AS6C1008-55PCN" H 8050 -400 50  0000 C TNN
-F 2 "" H 8000 1450 50  0001 L BNN
+F 2 "Housings_DIP:DIP-32_W15.24mm_Socket_LongPads" H 8000 1450 50  0001 L BNN
 F 3 "Alliance Memory" H 8000 1450 50  0001 L BNN
 F 4 "AS6C1008 Series 1-Mbit 128Kx8 55ns CMOS Static RAM" H 8000 1450 50  0001 L BNN "Description"
@@
 F 0 "C6" H 3875 7750 50  0000 L CNN
 F 1 "0.1uF" H 3875 7550 50  0000 L CNN
-F 2 "" H 3888 7500 50  0001 C CNN
+F 2 "Capacitors_THT:C_Disc_D4.3mm_W1.9mm_P5.00mm" H 3888 7500 50  0001 C CNN
 F 3 "" H 3850 7650 50  0001 C CNN
 	1    3850 7650
@@
 F 0 "C7" H 4175 7750 50  0000 L CNN
 F 1 "0.1uF" H 4175 7550 50  0000 L CNN
-F 2 "" H 4188 7500 50  0001 C CNN
+F 2 "Capacitors_THT:C_Disc_D4.3mm_W1.9mm_P5.00mm" H 4188 7500 50  0001 C CNN
 F 3 "" H 4150 7650 50  0001 C CNN
 	1    4150 7650
@@
 F 0 "U6" H 3650 5900 50  0000 C CNN
 F 1 "74AHC138" H 3700 4851 50  0000 C CNN
-F 2 "" H 3550 5400 50  0001 C CNN
+F 2 "Housings_DIP:DIP-16_W7.62mm_LongPads" H 3550 5400 50  0001 C CNN
 F 3 "" H 3550 5400 50  0001 C CNN
 	1    3550 5400
@@
 F 0 "D1" H 1300 4175 50  0000 L CNN
 F 1 "Green" H 1350 3952 50  0000 C CNN
-F 2 "" V 1350 4050 50  0001 C CNN
+F 2 "LEDs:LED_D5.0mm" V 1350 4050 50  0001 C CNN
 F 3 "" V 1350 4050 50  0001 C CNN
 	1    1350 4050
@@
 F 0 "R18" V 1430 4300 50  0000 C CNN
 F 1 "10K" V 1350 4300 50  0000 C CNN
-F 2 "" V 1280 4300 50  0001 C CNN
+F 2 "Resistors_THT:R_Axial_DIN0204_L3.6mm_D1.6mm_P5.08mm_Horizontal" V 1280 4300 50  0001 C CNN
 F 3 "" H 1350 4300 50  0001 C CNN
 	1    1350 4300
@@
 F 0 "J6" H 2100 4550 50  0000 C CNN
 F 1 "PWR" H 2100 4250 50  0000 C CNN
-F 2 "" H 2100 4450 50  0001 C CNN
+F 2 "Pin_Headers:Pin_Header_Straight_2x01_Pitch2.54mm" H 2100 4450 50  0001 C CNN
 F 3 "" H 2100 4450 50  0001 C CNN
 	1    2100 4450
@@
 F 0 "C24" H 1660 4220 50  0000 L CNN
 F 1 "10uF" H 1660 4070 50  0000 L CNN
-F 2 "" H 1650 4150 50  0001 C CNN
+F 2 "Capacitors_THT:C_Disc_D4.3mm_W1.9mm_P5.00mm" H 1650 4150 50  0001 C CNN
 F 3 "" H 1650 4150 50  0001 C CNN
 	1    1650 4150
@@
 F 0 "R29" V 2680 2250 50  0000 C CNN
 F 1 "10K" V 2600 2250 50  0000 C CNN
-F 2 "" V 2530 2250 50  0001 C CNN
+F 2 "Resistors_THT:R_Axial_DIN0204_L3.6mm_D1.6mm_P5.08mm_Horizontal" V 2530 2250 50  0001 C CNN
 F 3 "" H 2600 2250 50  0001 C CNN
 	1    2600 2250
@@
 F 0 "C26" H 4475 7750 50  0000 L CNN
 F 1 "0.1uF" H 4475 7550 50  0000 L CNN
-F 2 "" H 4488 7500 50  0001 C CNN
+F 2 "Capacitors_THT:C_Disc_D4.3mm_W1.9mm_P5.00mm" H 4488 7500 50  0001 C CNN
 F 3 "" H 4450 7650 50  0001 C CNN
 	1    4450 7650
@@
 F 0 "J5" H 600 4500 50  0000 L CNN
 F 1 "USB_B" H 600 4400 50  0000 L CNN
-F 2 "" H 950 4000 50  0001 C CNN
+F 2 "z80_footprints:USB_B_E8144-B02022-L" H 950 4000 50  0001 C CNN
 F 3 "" H 950 4000 50  0001 C CNN
 	1    800  4050
@@
 F 0 "U4" H 8850 900 50  0000 C CNN
 F 1 "74AHC32" H 8850 800 50  0000 C CNN
-F 2 "" H 8850 850 50  0001 C CNN
+F 2 "Housings_DIP:DIP-14_W7.62mm_LongPads" H 8850 850 50  0001 C CNN
 F 3 "" H 8850 850 50  0001 C CNN
 	3    8850 850
@@
 Wire Wire Line
 	9450 950  9600 950
-$Comp
-L Conn_02x20_Top_Bottom J3
-U 1 1 5ABBD7C9
-P 9750 2450
-F 0 "J3" H 9800 3450 50  0000 C CNN
-F 1 "Conn_02x20_Top_Bottom" H 9800 1350 50  0000 C CNN
-F 2 "" H 9750 2450 50  0001 C CNN
-F 3 "" H 9750 2450 50  0001 C CNN
-	1    9750 2450
-	1    0    0    -1
-$EndComp
 Wire Wire Line
 	9550 1550 9300 1550
@@
 NoConn ~ 10300 3050
 NoConn ~ 10300 3150
+$Comp
+L Conn_02x20_Odd_Even J3
+U 1 1 5AC5425B
+P 9750 2450
+F 0 "J3" H 9800 3450 50  0000 C CNN
+F 1 "Conn_02x20_Odd_Even" H 9800 1350 50  0000 C CNN
+F 2 "Pin_Headers:Pin_Header_Straight_2x20_Pitch2.54mm" H 9750 2450 50  0001 C CNN
+F 3 "" H 9750 2450 50  0001 C CNN
+	1    9750 2450
+	1    0    0    -1
+$EndComp
 $EndSCHEMATC

Commit message: Completed first pass of board layout.
git-svn-id: svn+ssh://dev.thehead.ca/depot/main/z80@618 995eaefb-0ce2-40e3-b8bc-69bf8729875b
Connections:
- net ~INT: now also J3.26 (Pin_26); no longer J3.39 (Pin_39)
Changed lines of the file:
@@
 Sheet 1 7
 Title "Z80 Prototype"
-Date "2018-04-11"
-Rev "7"
+Date "2018-05-09"
+Rev "8"
 Comp ""
 Comment1 ""
@@
 Text Label 9300 3350 0    60   ~ 0
 ~RESET
-Text Label 9300 3450 0    60   ~ 0
+Text Label 10300 2750 2    60   ~ 0
 ~INT
 Text Label 10300 3350 2    60   ~ 0
@@
 ~IORQ
 NoConn ~ 9300 3250
-NoConn ~ 10300 2750
 NoConn ~ 10300 2850
 NoConn ~ 10300 2950
@@
 	1    0    0    -1
 $EndComp
+Text Label 5200 4300 0    60   ~ 0
+D[0..7]
+NoConn ~ 9300 3450
 $EndSCHEMATC

Commit message: Initial prototype PCB build.
git-svn-id: svn+ssh://dev.thehead.ca/depot/main/z80@619 995eaefb-0ce2-40e3-b8bc-69bf8729875b
Connections:
- net ~IORQ5: now reaches U6.10 (O5)
- net ~IORQ5: now also J3.30 (Pin_30)
- net ~IORQ7: now reaches U6.7 (O7)
- net ~IORQ7: now also J3.28 (Pin_28)
- net ~IORQ6: now reaches U6.9 (O6)
- net ~IORQ6: now also J3.32 (Pin_32)
- no-connect marks 18 -> 12
Changed lines of the file:
@@
 Sheet 1 7
 Title "Z80 Prototype"
-Date "2018-05-09"
-Rev "8"
+Date "2018-05-23"
+Rev "9"
 Comp ""
 Comment1 ""
@@
 Wire Wire Line
 	7050 950  6900 950
-NoConn ~ 4150 5550
-NoConn ~ 4150 5650
-NoConn ~ 4150 5750
 $Comp
 L LED_Small_ALT D1
@@
 ~IORQ
 NoConn ~ 9300 3250
-NoConn ~ 10300 2850
-NoConn ~ 10300 2950
-NoConn ~ 10300 3050
 NoConn ~ 10300 3150
 $Comp
@@
 D[0..7]
 NoConn ~ 9300 3450
+Wire Wire Line
+	4150 5550 4450 5550
+Wire Wire Line
+	4150 5650 4450 5650
+Wire Wire Line
+	4150 5750 4450 5750
+Text Label 4450 5550 2    60   ~ 0
+~IORQ5
+Text Label 4450 5650 2    60   ~ 0
+~IORQ6
+Text Label 4450 5750 2    60   ~ 0
+~IORQ7
+Text Label 10300 2850 2    60   ~ 0
+~IORQ7
+Text Label 10300 2950 2    60   ~ 0
+~IORQ5
+Text Label 10300 3050 2    60   ~ 0
+~IORQ6
 $EndSCHEMATC

Commit message: Fix footprint for C24 to be a polarized radial electrolytic THT capacitor.
git-svn-id: svn+ssh://dev.thehead.ca/depot/main/z80@621 995eaefb-0ce2-40e3-b8bc-69bf8729875b
Parts:
- C24: footprint Capacitors_THT:C_Disc_D4.3mm_W1.9mm_P5.00mm -> Capacitors_THT:CP_Radial_D5.0mm_P2.50mm
Changed lines of the file:
@@
 F 0 "C24" H 1660 4220 50  0000 L CNN
 F 1 "10uF" H 1660 4070 50  0000 L CNN
-F 2 "Capacitors_THT:C_Disc_D4.3mm_W1.9mm_P5.00mm" H 1650 4150 50  0001 C CNN
+F 2 "Capacitors_THT:CP_Radial_D5.0mm_P2.50mm" H 1650 4150 50  0001 C CNN
 F 3 "" H 1650 4150 50  0001 C CNN
 	1    1650 4150
