File: z80.sch (KiCad schematic (older format))
At the start: 26 parts, among them J3 Conn_02x20_Odd_Even, J5 USB_B, J6 PWR, SW1 KS01Q, U1 Z80CPU, U2 74AHC14, U20 MIC5504-3.3YM5, U3 SST39SF010, U4 74AHC32, U5 AS6C1008-55PCN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

Commit message: Latest updates; preparing to move to github (I think).
git-svn-id: svn+ssh://dev.thehead.ca/depot/main/z80@636 995eaefb-0ce2-40e3-b8bc-69bf8729875b
Parts:
- removed unit 1 of U4
- removed unit 3 of U4
Connections:
- net A14: no longer U3.29 (A14), U5.3 (A14)
- net A15: no longer U3.3 (A15), U5.31 (A15)
- net GND: no longer U3.2 (A16), U5.2 (A16)
- net PA17: now reaches U4.5, U5.30 (CE2)
- new net PA14: U3.29 (A14), U5.3 (A14)
- new net PA15: U3.3 (A15), U5.31 (A15)
- new net PA16: U3.2 (A16), U5.2 (A16)
