File: 7-Segment Display.sch (KiCad schematic (older format))
At the start: 23 parts, among them U2 74AHC14, U4 74AHC32, U7 74AC574, U8 74AC574

Commit message: Latest rev of z80 schematic.
git-svn-id: svn+ssh://dev.thehead.ca/depot/main/z80@613 995eaefb-0ce2-40e3-b8bc-69bf8729875b
Parts:
- removed U2: 74AHC14, symbol 74HC14
- removed U4: 74AHC32, symbol 74LS32
- added C20: 0.1uF, symbol C
- added U9: 74AHC02, symbol 74HC02
Connections:
- net GND: now also C20.2, U9.7 (GND), U9.7 (GND)
- net VCC: now also C20.1, U9.14 (VCC), U9.14 (VCC)
- net ~IORQ0: now also U9.3
- net ~IORQ1: now also U9.6
- net ~WR: now also U9.2, U9.5
- net at U7.11 (Cp): now also U9.1
- net at U8.11 (Cp): now also U9.4
Other:
- note added: "Near\nU9"
Changed lines of the file:
@@
 $Descr USLetter 11000 8500
 encoding utf-8
-Sheet 3 6
+Sheet 3 7
 Title "7-Segment Display"
-Date "2017-10-22"
-Rev "4"
+Date "2017-10-24"
+Rev "5"
 Comp ""
 Comment1 ""
@@
 $EndDescr
 $Comp
-L 74HC14 U2
-U 3 1 59D6D678
-P 4100 3600
-F 0 "U2" H 4250 3700 50  0000 C CNN
-F 1 "74AHC14" H 4300 3500 50  0000 C CNN
-F 2 "" H 4100 3600 50  0001 C CNN
-F 3 "" H 4100 3600 50  0001 C CNN
-	3    4100 3600
-	1    0    0    -1
-$EndComp
-$Comp
-L 74HC14 U2
-U 4 1 59D6D67F
-P 4100 4900
-F 0 "U2" H 4250 5000 50  0000 C CNN
-F 1 "74AHC14" H 4300 4800 50  0000 C CNN
-F 2 "" H 4100 4900 50  0001 C CNN
-F 3 "" H 4100 4900 50  0001 C CNN
-	4    4100 4900
-	1    0    0    -1
-$EndComp
-$Comp
-L 74LS32 U4
-U 3 1 59D6D686
-P 3050 3600
-F 0 "U4" H 3050 3650 50  0000 C CNN
-F 1 "74AHC32" H 3050 3550 50  0000 C CNN
-F 2 "" H 3050 3600 50  0001 C CNN
-F 3 "" H 3050 3600 50  0001 C CNN
-	3    3050 3600
-	1    0    0    -1
-$EndComp
-$Comp
-L 74LS32 U4
-U 4 1 59D6D68D
-P 3050 4900
-F 0 "U4" H 3050 4950 50  0000 C CNN
-F 1 "74AHC32" H 3050 4850 50  0000 C CNN
-F 2 "" H 3050 4900 50  0001 C CNN
-F 3 "" H 3050 4900 50  0001 C CNN
-	4    3050 4900
-	1    0    0    -1
-$EndComp
-$Comp
-L GND #PWR031
+L GND #PWR030
 U 1 1 59D6D694
 P 4650 3700
-F 0 "#PWR031" H 4650 3450 50  0001 C CNN
+F 0 "#PWR030" H 4650 3450 50  0001 C CNN
 F 1 "GND" H 4650 3550 50  0000 C CNN
 F 2 "" H 4650 3700 50  0001 C CNN
@@
 $EndComp
 $Comp
-L GND #PWR032
+L GND #PWR031
 U 1 1 59D6D6E9
 P 4650 5000
-F 0 "#PWR032" H 4650 4750 50  0001 C CNN
+F 0 "#PWR031" H 4650 4750 50  0001 C CNN
 F 1 "GND" H 4650 4850 50  0000 C CNN
 F 2 "" H 4650 5000 50  0001 C CNN
@@
 	8600 4700 6450 4700
 $Comp
-L GND #PWR033
+L GND #PWR032
 U 1 1 59D6D771
 P 8400 2600
-F 0 "#PWR033" H 8400 2350 50  0001 C CNN
+F 0 "#PWR032" H 8400 2350 50  0001 C CNN
 F 1 "GND" H 8400 2450 50  0000 C CNN
 F 2 "" H 8400 2600 50  0001 C CNN
@@
 	8400 2400 8400 2600
 Wire Wire Line
-	4750 3600 4550 3600
-Wire Wire Line
-	4550 4900 4750 4900
-Wire Wire Line
-	1450 3500 2450 3500
-Wire Wire Line
-	2050 4800 2450 4800
-Wire Wire Line
-	1450 3700 2450 3700
-Wire Wire Line
-	1450 5000 2450 5000
+	4400 3600 4750 3600
+Wire Wire Line
+	4400 4900 4750 4900
+Wire Wire Line
+	1450 3500 3200 3500
+Wire Wire Line
+	2050 4800 3200 4800
+Wire Wire Line
+	1450 3700 3200 3700
+Wire Wire Line
+	1450 5000 3200 5000
 Text HLabel 1450 2250 0    60   BiDi ~ 0
 D[0..7]
@@
 $EndComp
 $Comp
-L GND #PWR034
+L GND #PWR033
 U 1 1 59D81B6F
 P 5200 1550
-F 0 "#PWR034" H 5200 1300 50  0001 C CNN
+F 0 "#PWR033" H 5200 1300 50  0001 C CNN
 F 1 "GND" H 5200 1400 50  0000 C CNN
 F 2 "" H 5200 1550 50  0001 C CNN
@@
 $EndComp
 $Comp
-L VCC #PWR035
+L VCC #PWR034
 U 1 1 59D81B7C
 P 5200 1250
-F 0 "#PWR035" H 5200 1100 50  0001 C CNN
+F 0 "#PWR034" H 5200 1100 50  0001 C CNN
 F 1 "VCC" H 5200 1400 50  0000 C CNN
 F 2 "" H 5200 1250 50  0001 C CNN
@@
 Connection ~ 5750 1550
 Wire Wire Line
-	5200 1550 5750 1550
-Wire Wire Line
-	5200 1250 5750 1250
+	5200 1550 6050 1550
+Wire Wire Line
+	5200 1250 6050 1250
+$Comp
+L 74HC02 U9
+U 1 1 59EFCF09
+P 3800 3600
+F 0 "U9" H 3800 3650 50  0000 C CNN
+F 1 "74AHC02" H 3850 3550 50  0000 C CNN
+F 2 "" H 3800 3600 50  0001 C CNN
+F 3 "" H 3800 3600 50  0001 C CNN
+	1    3800 3600
+	1    0    0    -1
+$EndComp
+$Comp
+L 74HC02 U9
+U 2 1 59EFD198
+P 3800 4900
+F 0 "U9" H 3800 4950 50  0000 C CNN
+F 1 "74AHC02" H 3850 4850 50  0000 C CNN
+F 2 "" H 3800 4900 50  0001 C CNN
+F 3 "" H 3800 4900 50  0001 C CNN
+	2    3800 4900
+	1    0    0    -1
+$EndComp
+$Comp
+L C C20
+U 1 1 59EFD5EA
+P 6050 1400
+F 0 "C20" H 6075 1500 50  0000 L CNN
+F 1 "0.1uF" H 6075 1300 50  0000 L CNN
+F 2 "" H 6088 1250 50  0001 C CNN
+F 3 "" H 6050 1400 50  0001 C CNN
+	1    6050 1400
+	1    0    0    -1
+$EndComp
+Text Notes 6000 1200 0    60   ~ 0
+Near\nU9
 $EndSCHEMATC

Commit message: Assign footprints to schematic, drawing custom connector, socket, and switch footprints as needed.
git-svn-id: svn+ssh://dev.thehead.ca/depot/main/z80@617 995eaefb-0ce2-40e3-b8bc-69bf8729875b
Parts:
- AFF1: footprint (none) -> z80_footprints:LTD-6940HR
- C10, C11, C20: footprint (none) -> Capacitors_THT:C_Disc_D4.3mm_W1.9mm_P5.00mm
- R12, R13, R14, R15, R16, R17, R19, R20, R21, R22, R23, R24, R25, R26, R27, R28: footprint (none) -> Resistors_THT:R_Axial_DIN0204_L3.6mm_D1.6mm_P5.08mm_Horizontal
- U7, U8: footprint (none) -> Housings_DIP:DIP-20_W7.62mm_LongPads
- U9: footprint (none) -> Housings_DIP:DIP-14_W7.62mm_LongPads
Changed lines of the file:
@@
 Sheet 3 7
 Title "7-Segment Display"
-Date "2018-03-28"
-Rev "6"
+Date "2018-04-11"
+Rev "7"
 Comp ""
 Comment1 ""
@@
 F 0 "U7" H 5450 3200 50  0000 C CNN
 F 1 "74AC574" H 5500 2850 50  0000 C CNN
-F 2 "" H 5450 3200 50  0001 C CNN
+F 2 "Housings_DIP:DIP-20_W7.62mm_LongPads" H 5450 3200 50  0001 C CNN
 F 3 "" H 5450 3200 50  0001 C CNN
 	1    5450 3200
@@
 F 0 "R12" V 6261 2810 50  0000 L CNN
 F 1 "220R" V 6300 2700 50  0000 C CNN
-F 2 "" V 6230 2700 50  0001 C CNN
+F 2 "Resistors_THT:R_Axial_DIN0204_L3.6mm_D1.6mm_P5.08mm_Horizontal" V 6230 2700 50  0001 C CNN
 F 3 "" H 6300 2700 50  0001 C CNN
 	1    6300 2700
@@
 F 0 "R13" V 6261 2910 50  0000 L CNN
 F 1 "220R" V 6300 2800 50  0000 C CNN
-F 2 "" V 6230 2800 50  0001 C CNN
+F 2 "Resistors_THT:R_Axial_DIN0204_L3.6mm_D1.6mm_P5.08mm_Horizontal" V 6230 2800 50  0001 C CNN
 F 3 "" H 6300 2800 50  0001 C CNN
 	1    6300 2800
@@
 F 0 "R14" V 6261 3010 50  0000 L CNN
 F 1 "220R" V 6300 2900 50  0000 C CNN
-F 2 "" V 6230 2900 50  0001 C CNN
+F 2 "Resistors_THT:R_Axial_DIN0204_L3.6mm_D1.6mm_P5.08mm_Horizontal" V 6230 2900 50  0001 C CNN
 F 3 "" H 6300 2900 50  0001 C CNN
 	1    6300 2900
@@
 F 0 "R15" V 6261 3110 50  0000 L CNN
 F 1 "220R" V 6300 3000 50  0000 C CNN
-F 2 "" V 6230 3000 50  0001 C CNN
+F 2 "Resistors_THT:R_Axial_DIN0204_L3.6mm_D1.6mm_P5.08mm_Horizontal" V 6230 3000 50  0001 C CNN
 F 3 "" H 6300 3000 50  0001 C CNN
 	1    6300 3000
@@
 F 0 "R16" V 6261 3210 50  0000 L CNN
 F 1 "220R" V 6300 3100 50  0000 C CNN
-F 2 "" V 6230 3100 50  0001 C CNN
+F 2 "Resistors_THT:R_Axial_DIN0204_L3.6mm_D1.6mm_P5.08mm_Horizontal" V 6230 3100 50  0001 C CNN
 F 3 "" H 6300 3100 50  0001 C CNN
 	1    6300 3100
@@
 F 0 "R17" V 6261 3310 50  0000 L CNN
 F 1 "220R" V 6300 3200 50  0000 C CNN
-F 2 "" V 6230 3200 50  0001 C CNN
+F 2 "Resistors_THT:R_Axial_DIN0204_L3.6mm_D1.6mm_P5.08mm_Horizontal" V 6230 3200 50  0001 C CNN
 F 3 "" H 6300 3200 50  0001 C CNN
 	1    6300 3200
@@
 F 0 "R19" V 6261 3410 50  0000 L CNN
 F 1 "220R" V 6300 3300 50  0000 C CNN
-F 2 "" V 6230 3300 50  0001 C CNN
+F 2 "Resistors_THT:R_Axial_DIN0204_L3.6mm_D1.6mm_P5.08mm_Horizontal" V 6230 3300 50  0001 C CNN
 F 3 "" H 6300 3300 50  0001 C CNN
 	1    6300 3300
@@
 F 0 "R20" V 6261 3510 50  0000 L CNN
 F 1 "220R" V 6300 3400 50  0000 C CNN
-F 2 "" V 6230 3400 50  0001 C CNN
+F 2 "Resistors_THT:R_Axial_DIN0204_L3.6mm_D1.6mm_P5.08mm_Horizontal" V 6230 3400 50  0001 C CNN
 F 3 "" H 6300 3400 50  0001 C CNN
 	1    6300 3400
@@
 F 0 "U8" H 5450 4500 50  0000 C CNN
 F 1 "74AC574" H 5500 4150 50  0000 C CNN
-F 2 "" H 5450 4500 50  0001 C CNN
+F 2 "Housings_DIP:DIP-20_W7.62mm_LongPads" H 5450 4500 50  0001 C CNN
 F 3 "" H 5450 4500 50  0001 C CNN
 	1    5450 4500
@@
 F 0 "R21" V 6261 4110 50  0000 L CNN
 F 1 "220R" V 6300 4000 50  0000 C CNN
-F 2 "" V 6230 4000 50  0001 C CNN
+F 2 "Resistors_THT:R_Axial_DIN0204_L3.6mm_D1.6mm_P5.08mm_Horizontal" V 6230 4000 50  0001 C CNN
 F 3 "" H 6300 4000 50  0001 C CNN
 	1    6300 4000
@@
 F 0 "R22" V 6261 4210 50  0000 L CNN
 F 1 "220R" V 6300 4100 50  0000 C CNN
-F 2 "" V 6230 4100 50  0001 C CNN
+F 2 "Resistors_THT:R_Axial_DIN0204_L3.6mm_D1.6mm_P5.08mm_Horizontal" V 6230 4100 50  0001 C CNN
 F 3 "" H 6300 4100 50  0001 C CNN
 	1    6300 4100
@@
 F 0 "R23" V 6261 4310 50  0000 L CNN
 F 1 "220R" V 6300 4200 50  0000 C CNN
-F 2 "" V 6230 4200 50  0001 C CNN
+F 2 "Resistors_THT:R_Axial_DIN0204_L3.6mm_D1.6mm_P5.08mm_Horizontal" V 6230 4200 50  0001 C CNN
 F 3 "" H 6300 4200 50  0001 C CNN
 	1    6300 4200
@@
 F 0 "R24" V 6261 4410 50  0000 L CNN
 F 1 "220R" V 6300 4300 50  0000 C CNN
-F 2 "" V 6230 4300 50  0001 C CNN
+F 2 "Resistors_THT:R_Axial_DIN0204_L3.6mm_D1.6mm_P5.08mm_Horizontal" V 6230 4300 50  0001 C CNN
 F 3 "" H 6300 4300 50  0001 C CNN
 	1    6300 4300
@@
 F 0 "R25" V 6261 4510 50  0000 L CNN
 F 1 "220R" V 6300 4400 50  0000 C CNN
-F 2 "" V 6230 4400 50  0001 C CNN
+F 2 "Resistors_THT:R_Axial_DIN0204_L3.6mm_D1.6mm_P5.08mm_Horizontal" V 6230 4400 50  0001 C CNN
 F 3 "" H 6300 4400 50  0001 C CNN
 	1    6300 4400
@@
 F 0 "R26" V 6261 4610 50  0000 L CNN
 F 1 "220R" V 6300 4500 50  0000 C CNN
-F 2 "" V 6230 4500 50  0001 C CNN
+F 2 "Resistors_THT:R_Axial_DIN0204_L3.6mm_D1.6mm_P5.08mm_Horizontal" V 6230 4500 50  0001 C CNN
 F 3 "" H 6300 4500 50  0001 C CNN
 	1    6300 4500
@@
 F 0 "R27" V 6261 4710 50  0000 L CNN
 F 1 "220R" V 6300 4600 50  0000 C CNN
-F 2 "" V 6230 4600 50  0001 C CNN
+F 2 "Resistors_THT:R_Axial_DIN0204_L3.6mm_D1.6mm_P5.08mm_Horizontal" V 6230 4600 50  0001 C CNN
 F 3 "" H 6300 4600 50  0001 C CNN
 	1    6300 4600
@@
 F 0 "R28" V 6261 4810 50  0000 L CNN
 F 1 "220R" V 6300 4700 50  0000 C CNN
-F 2 "" V 6230 4700 50  0001 C CNN
+F 2 "Resistors_THT:R_Axial_DIN0204_L3.6mm_D1.6mm_P5.08mm_Horizontal" V 6230 4700 50  0001 C CNN
 F 3 "" H 6300 4700 50  0001 C CNN
 	1    6300 4700
@@
 F 0 "AFF1" H 7350 3550 50  0000 C CNN
 F 1 "LTD-6940HR" H 7350 2450 50  0000 C CNN
-F 2 "" H 7100 3000 50  0001 C CNN
+F 2 "z80_footprints:LTD-6940HR" H 7100 3000 50  0001 C CNN
 F 3 "https://media.digikey.com/pdf/Data%20Sheets/Lite-On%20PDFs/LTD-6000_Series.pdf" H 7100 2291 50  0001 C CNN
 	1    7350 3000
@@
 F 0 "C10" H 5475 1500 50  0000 L CNN
 F 1 "0.1uF" H 5475 1300 50  0000 L CNN
-F 2 "" H 5488 1250 50  0001 C CNN
+F 2 "Capacitors_THT:C_Disc_D4.3mm_W1.9mm_P5.00mm" H 5488 1250 50  0001 C CNN
 F 3 "" H 5450 1400 50  0001 C CNN
 	1    5450 1400
@@
 F 0 "C11" H 5775 1500 50  0000 L CNN
 F 1 "0.1uF" H 5775 1300 50  0000 L CNN
-F 2 "" H 5788 1250 50  0001 C CNN
+F 2 "Capacitors_THT:C_Disc_D4.3mm_W1.9mm_P5.00mm" H 5788 1250 50  0001 C CNN
 F 3 "" H 5750 1400 50  0001 C CNN
 	1    5750 1400
@@
 F 0 "U9" H 3800 3650 50  0000 C CNN
 F 1 "74AHC02" H 3850 3550 50  0000 C CNN
-F 2 "" H 3800 3600 50  0001 C CNN
+F 2 "Housings_DIP:DIP-14_W7.62mm_LongPads" H 3800 3600 50  0001 C CNN
 F 3 "" H 3800 3600 50  0001 C CNN
 	1    3800 3600
@@
 F 0 "U9" H 3800 4950 50  0000 C CNN
 F 1 "74AHC02" H 3850 4850 50  0000 C CNN
-F 2 "" H 3800 4900 50  0001 C CNN
+F 2 "Housings_DIP:DIP-14_W7.62mm_LongPads" H 3800 4900 50  0001 C CNN
 F 3 "" H 3800 4900 50  0001 C CNN
 	2    3800 4900
@@
 F 0 "C20" H 6075 1500 50  0000 L CNN
 F 1 "0.1uF" H 6075 1300 50  0000 L CNN
-F 2 "" H 6088 1250 50  0001 C CNN
+F 2 "Capacitors_THT:C_Disc_D4.3mm_W1.9mm_P5.00mm" H 6088 1250 50  0001 C CNN
 F 3 "" H 6050 1400 50  0001 C CNN
 	1    6050 1400
