File: CTC.sch (KiCad schematic (older format))
At the start: 3 parts, among them U17 Z84C30, X2 1.8432MHz

Commit message: Assign footprints to schematic, drawing custom connector, socket, and switch footprints as needed.
git-svn-id: svn+ssh://dev.thehead.ca/depot/main/z80@617 995eaefb-0ce2-40e3-b8bc-69bf8729875b
Parts:
- C27: footprint (none) -> Capacitors_THT:C_Disc_D4.3mm_W1.9mm_P5.00mm
- U17: footprint (none) -> z80_footprints:8444-11B1-RK-TP
Changed lines of the file:
@@
 Sheet 6 7
 Title "CTC, Baud Rate Generation"
-Date "2018-03-28"
-Rev "6"
+Date "2018-04-11"
+Rev "7"
 Comp ""
 Comment1 ""
@@
 F 0 "U17" H 3000 4241 50  0000 L TNN
 F 1 "Z84C30" H 4000 4250 50  0000 R TNN
-F 2 "" H 4000 4250 60  0001 C CNN
+F 2 "z80_footprints:8444-11B1-RK-TP" H 4000 4250 60  0001 C CNN
 F 3 "" H 4000 4250 60  0001 C CNN
 	1    3500 3150
@@
 $EndComp
 $Comp
-L VCC #PWR065
+L VCC #PWR066
 U 1 1 59D9205A
 P 3500 1950
-F 0 "#PWR065" H 3500 1800 50  0001 C CNN
+F 0 "#PWR066" H 3500 1800 50  0001 C CNN
 F 1 "VCC" H 3500 2100 50  0000 C CNN
 F 2 "" H 3500 1950 50  0001 C CNN
@@
 $EndComp
 $Comp
-L GND #PWR066
+L GND #PWR067
 U 1 1 59D92070
 P 3500 4950
-F 0 "#PWR066" H 3500 4700 50  0001 C CNN
+F 0 "#PWR067" H 3500 4700 50  0001 C CNN
 F 1 "GND" H 3500 4800 50  0000 C CNN
 F 2 "" H 3500 4950 50  0001 C CNN
@@
 F 0 "C27" H 4825 6850 50  0000 L CNN
 F 1 "0.1uF" H 4825 6650 50  0000 L CNN
-F 2 "" H 4838 6600 50  0001 C CNN
+F 2 "Capacitors_THT:C_Disc_D4.3mm_W1.9mm_P5.00mm" H 4838 6600 50  0001 C CNN
 F 3 "" H 4800 6750 50  0001 C CNN
 	1    4800 6750
@@
 $EndComp
 $Comp
-L GND #PWR067
+L GND #PWR068
 U 1 1 59D92BA2
 P 4550 6900
-F 0 "#PWR067" H 4550 6650 50  0001 C CNN
+F 0 "#PWR068" H 4550 6650 50  0001 C CNN
 F 1 "GND" H 4550 6750 50  0000 C CNN
 F 2 "" H 4550 6900 50  0001 C CNN
@@
 $EndComp
 $Comp
-L VCC #PWR068
+L VCC #PWR069
 U 1 1 59D92BAF
 P 4550 6600
-F 0 "#PWR068" H 4550 6450 50  0001 C CNN
+F 0 "#PWR069" H 4550 6450 50  0001 C CNN
 F 1 "VCC" H 4550 6750 50  0000 C CNN
 F 2 "" H 4550 6600 50  0001 C CNN
@@
 $EndComp
 $Comp
-L GND #PWR069
+L GND #PWR070
 U 1 1 59DCF0C9
 P 5500 2550
-F 0 "#PWR069" H 5500 2300 50  0001 C CNN
+F 0 "#PWR070" H 5500 2300 50  0001 C CNN
 F 1 "GND" H 5500 2400 50  0000 C CNN
 F 2 "" H 5500 2550 50  0001 C CNN
@@
 $EndComp
 $Comp
-L VCC #PWR070
+L VCC #PWR071
 U 1 1 59DCF0CF
 P 5500 1950
-F 0 "#PWR070" H 5500 1800 50  0001 C CNN
+F 0 "#PWR071" H 5500 1800 50  0001 C CNN
 F 1 "VCC" H 5500 2100 50  0000 C CNN
 F 2 "" H 5500 1950 50  0001 C CNN
