File: joystick.sch (KiCad schematic (older format))
At the start: 16 parts, among them U13 74AHC541, U14 74AHC541

Commit message: Assign footprints to schematic, drawing custom connector, socket, and switch footprints as needed.
git-svn-id: svn+ssh://dev.thehead.ca/depot/main/z80@617 995eaefb-0ce2-40e3-b8bc-69bf8729875b
Parts:
- C8, C9: footprint (none) -> Capacitors_THT:C_Disc_D4.3mm_W1.9mm_P5.00mm
- JOY1, JOY2: footprint (none) -> z80_footprints:L717SDE09P1ACH
- R10, R11, R2, R3, R4, R5, R6, R7, R8, R9: footprint (none) -> Resistors_THT:R_Axial_DIN0204_L3.6mm_D1.6mm_P5.08mm_Horizontal
- U13, U14: footprint (none) -> Housings_DIP:DIP-20_W7.62mm_LongPads
Changed lines of the file:
@@
 Sheet 2 7
 Title "Joystick Ports"
-Date "2018-03-28"
-Rev "6"
+Date "2018-04-11"
+Rev "7"
 Comp ""
 Comment1 ""
@@
 F 0 "U13" H 4650 3575 50  0000 C BNN
 F 1 "74AHC541" H 4650 2425 50  0000 C TNN
-F 2 "" H 4650 3000 50  0001 C CNN
+F 2 "Housings_DIP:DIP-20_W7.62mm_LongPads" H 4650 3000 50  0001 C CNN
 F 3 "" H 4650 3000 50  0001 C CNN
 	1    4650 3000
@@
 F 0 "JOY1" H 7050 3400 50  0000 C CNN
 F 1 "DB9-M" H 7050 3325 50  0000 C CNN
-F 2 "" H 7050 2750 50  0001 C CNN
+F 2 "z80_footprints:L717SDE09P1ACH" H 7050 2750 50  0001 C CNN
 F 3 "" H 7050 2750 50  0001 C CNN
 	1    7050 2750
@@
 F 0 "R2" V 5530 2250 50  0000 C CNN
 F 1 "10K" V 5450 2250 50  0000 C CNN
-F 2 "" V 5380 2250 50  0001 C CNN
+F 2 "Resistors_THT:R_Axial_DIN0204_L3.6mm_D1.6mm_P5.08mm_Horizontal" V 5380 2250 50  0001 C CNN
 F 3 "" H 5450 2250 50  0001 C CNN
 	1    5450 2250
@@
 F 0 "R4" V 5730 2250 50  0000 C CNN
 F 1 "10K" V 5650 2250 50  0000 C CNN
-F 2 "" V 5580 2250 50  0001 C CNN
+F 2 "Resistors_THT:R_Axial_DIN0204_L3.6mm_D1.6mm_P5.08mm_Horizontal" V 5580 2250 50  0001 C CNN
 F 3 "" H 5650 2250 50  0001 C CNN
 	1    5650 2250
@@
 F 0 "R6" V 5930 2250 50  0000 C CNN
 F 1 "10K" V 5850 2250 50  0000 C CNN
-F 2 "" V 5780 2250 50  0001 C CNN
+F 2 "Resistors_THT:R_Axial_DIN0204_L3.6mm_D1.6mm_P5.08mm_Horizontal" V 5780 2250 50  0001 C CNN
 F 3 "" H 5850 2250 50  0001 C CNN
 	1    5850 2250
@@
 F 0 "R8" V 6130 2250 50  0000 C CNN
 F 1 "10K" V 6050 2250 50  0000 C CNN
-F 2 "" V 5980 2250 50  0001 C CNN
+F 2 "Resistors_THT:R_Axial_DIN0204_L3.6mm_D1.6mm_P5.08mm_Horizontal" V 5980 2250 50  0001 C CNN
 F 3 "" H 6050 2250 50  0001 C CNN
 	1    6050 2250
@@
 F 0 "R10" V 6330 2250 50  0000 C CNN
 F 1 "10K" V 6250 2250 50  0000 C CNN
-F 2 "" V 6180 2250 50  0001 C CNN
+F 2 "Resistors_THT:R_Axial_DIN0204_L3.6mm_D1.6mm_P5.08mm_Horizontal" V 6180 2250 50  0001 C CNN
 F 3 "" H 6250 2250 50  0001 C CNN
 	1    6250 2250
@@
 F 0 "U14" H 4650 5275 50  0000 C BNN
 F 1 "74AHC541" H 4650 4125 50  0000 C TNN
-F 2 "" H 4650 4700 50  0001 C CNN
+F 2 "Housings_DIP:DIP-20_W7.62mm_LongPads" H 4650 4700 50  0001 C CNN
 F 3 "" H 4650 4700 50  0001 C CNN
 	1    4650 4700
@@
 F 0 "JOY2" H 7050 5100 50  0000 C CNN
 F 1 "DB9-M" H 7050 5025 50  0000 C CNN
-F 2 "" H 7050 4450 50  0001 C CNN
+F 2 "z80_footprints:L717SDE09P1ACH" H 7050 4450 50  0001 C CNN
 F 3 "" H 7050 4450 50  0001 C CNN
 	1    7050 4450
@@
 F 0 "R3" V 5530 3950 50  0000 C CNN
 F 1 "10K" V 5450 3950 50  0000 C CNN
-F 2 "" V 5380 3950 50  0001 C CNN
+F 2 "Resistors_THT:R_Axial_DIN0204_L3.6mm_D1.6mm_P5.08mm_Horizontal" V 5380 3950 50  0001 C CNN
 F 3 "" H 5450 3950 50  0001 C CNN
 	1    5450 3950
@@
 F 0 "R5" V 5730 3950 50  0000 C CNN
 F 1 "10K" V 5650 3950 50  0000 C CNN
-F 2 "" V 5580 3950 50  0001 C CNN
+F 2 "Resistors_THT:R_Axial_DIN0204_L3.6mm_D1.6mm_P5.08mm_Horizontal" V 5580 3950 50  0001 C CNN
 F 3 "" H 5650 3950 50  0001 C CNN
 	1    5650 3950
@@
 F 0 "R7" V 5930 3950 50  0000 C CNN
 F 1 "10K" V 5850 3950 50  0000 C CNN
-F 2 "" V 5780 3950 50  0001 C CNN
+F 2 "Resistors_THT:R_Axial_DIN0204_L3.6mm_D1.6mm_P5.08mm_Horizontal" V 5780 3950 50  0001 C CNN
 F 3 "" H 5850 3950 50  0001 C CNN
 	1    5850 3950
@@
 F 0 "R9" V 6130 3950 50  0000 C CNN
 F 1 "10K" V 6050 3950 50  0000 C CNN
-F 2 "" V 5980 3950 50  0001 C CNN
+F 2 "Resistors_THT:R_Axial_DIN0204_L3.6mm_D1.6mm_P5.08mm_Horizontal" V 5980 3950 50  0001 C CNN
 F 3 "" H 6050 3950 50  0001 C CNN
 	1    6050 3950
@@
 F 0 "R11" V 6330 3950 50  0000 C CNN
 F 1 "10K" V 6250 3950 50  0000 C CNN
-F 2 "" V 6180 3950 50  0001 C CNN
+F 2 "Resistors_THT:R_Axial_DIN0204_L3.6mm_D1.6mm_P5.08mm_Horizontal" V 6180 3950 50  0001 C CNN
 F 3 "" H 6250 3950 50  0001 C CNN
 	1    6250 3950
@@
 F 0 "C8" H 5175 1450 50  0000 L CNN
 F 1 "0.1uF" H 5175 1250 50  0000 L CNN
-F 2 "" H 5188 1200 50  0001 C CNN
+F 2 "Capacitors_THT:C_Disc_D4.3mm_W1.9mm_P5.00mm" H 5188 1200 50  0001 C CNN
 F 3 "" H 5150 1350 50  0001 C CNN
 	1    5150 1350
@@
 F 0 "C9" H 5475 1450 50  0000 L CNN
 F 1 "0.1uF" H 5475 1250 50  0000 L CNN
-F 2 "" H 5488 1200 50  0001 C CNN
+F 2 "Capacitors_THT:C_Disc_D4.3mm_W1.9mm_P5.00mm" H 5488 1200 50  0001 C CNN
 F 3 "" H 5450 1350 50  0001 C CNN
 	1    5450 1350
