File: spares.sch (KiCad schematic (older format))
At the start: 4 parts, among them U16 74AHC08, U2 74AHC14, U4 74AHC32, U9 74AHC02

Commit message: Assign footprints to schematic, drawing custom connector, socket, and switch footprints as needed.
git-svn-id: svn+ssh://dev.thehead.ca/depot/main/z80@617 995eaefb-0ce2-40e3-b8bc-69bf8729875b
Parts:
- U16, U2, U4, U9: footprint (none) -> Housings_DIP:DIP-14_W7.62mm_LongPads
Changed lines of the file:
@@
 Sheet 7 7
 Title ""
-Date "2018-03-28"
-Rev "6"
+Date "2018-04-11"
+Rev "7"
 Comp ""
 Comment1 ""
@@
 $EndDescr
 $Comp
-L GND #PWR071
+L GND #PWR072
 U 1 1 59EFCC3B
 P 800 2350
-F 0 "#PWR071" H 800 2100 50  0001 C CNN
+F 0 "#PWR072" H 800 2100 50  0001 C CNN
 F 1 "GND" H 800 2200 50  0000 C CNN
 F 2 "" H 800 2350 50  0001 C CNN
@@
 F 0 "U16" H 1400 1000 50  0000 C CNN
 F 1 "74AHC08" H 1400 900 50  0000 C CNN
-F 2 "" H 1400 950 50  0001 C CNN
+F 2 "Housings_DIP:DIP-14_W7.62mm_LongPads" H 1400 950 50  0001 C CNN
 F 3 "" H 1400 950 50  0001 C CNN
 	2    1400 950
@@
 F 0 "U16" H 1400 1450 50  0000 C CNN
 F 1 "74AHC08" H 1400 1350 50  0000 C CNN
-F 2 "" H 1400 1400 50  0001 C CNN
+F 2 "Housings_DIP:DIP-14_W7.62mm_LongPads" H 1400 1400 50  0001 C CNN
 F 3 "" H 1400 1400 50  0001 C CNN
 	3    1400 1400
@@
 F 0 "U16" H 1400 1950 50  0000 C CNN
 F 1 "74AHC08" H 1400 1850 50  0000 C CNN
-F 2 "" H 1400 1900 50  0001 C CNN
+F 2 "Housings_DIP:DIP-14_W7.62mm_LongPads" H 1400 1900 50  0001 C CNN
 F 3 "" H 1400 1900 50  0001 C CNN
 	4    1400 1900
@@
 F 0 "U2" H 4600 950 50  0000 C CNN
 F 1 "74AHC14" H 4650 750 50  0000 C CNN
-F 2 "" H 4450 850 50  0001 C CNN
+F 2 "Housings_DIP:DIP-14_W7.62mm_LongPads" H 4450 850 50  0001 C CNN
 F 3 "" H 4450 850 50  0001 C CNN
 	3    4450 850
@@
 F 0 "U2" H 4600 1350 50  0000 C CNN
 F 1 "74AHC14" H 4650 1150 50  0000 C CNN
-F 2 "" H 4450 1250 50  0001 C CNN
+F 2 "Housings_DIP:DIP-14_W7.62mm_LongPads" H 4450 1250 50  0001 C CNN
 F 3 "" H 4450 1250 50  0001 C CNN
 	4    4450 1250
@@
 F 0 "U4" H 3000 1000 50  0000 C CNN
 F 1 "74AHC32" H 3000 900 50  0000 C CNN
-F 2 "" H 3000 950 50  0001 C CNN
+F 2 "Housings_DIP:DIP-14_W7.62mm_LongPads" H 3000 950 50  0001 C CNN
 F 3 "" H 3000 950 50  0001 C CNN
 	4    3000 950
@@
 NoConn ~ 3600 950
 $Comp
-L GND #PWR072
+L GND #PWR073
 U 1 1 59EFDA1E
 P 2400 1350
-F 0 "#PWR072" H 2400 1100 50  0001 C CNN
+F 0 "#PWR073" H 2400 1100 50  0001 C CNN
 F 1 "GND" H 2400 1200 50  0000 C CNN
 F 2 "" H 2400 1350 50  0001 C CNN
@@
 $EndComp
 $Comp
-L GND #PWR073
+L GND #PWR074
 U 1 1 59EFDA40
 P 4000 1600
-F 0 "#PWR073" H 4000 1350 50  0001 C CNN
+F 0 "#PWR074" H 4000 1350 50  0001 C CNN
 F 1 "GND" H 4000 1450 50  0000 C CNN
 F 2 "" H 4000 1600 50  0001 C CNN
@@
 F 0 "U9" H 6000 1000 50  0000 C CNN
 F 1 "74AHC02" H 6050 900 50  0000 C CNN
-F 2 "" H 6000 950 50  0001 C CNN
+F 2 "Housings_DIP:DIP-14_W7.62mm_LongPads" H 6000 950 50  0001 C CNN
 F 3 "" H 6000 950 50  0001 C CNN
 	3    6000 950
@@
 F 0 "U9" H 6000 1450 50  0000 C CNN
 F 1 "74AHC02" H 6050 1350 50  0000 C CNN
-F 2 "" H 6000 1400 50  0001 C CNN
+F 2 "Housings_DIP:DIP-14_W7.62mm_LongPads" H 6000 1400 50  0001 C CNN
 F 3 "" H 6000 1400 50  0001 C CNN
 	4    6000 1400
@@
 NoConn ~ 6600 1400
 $Comp
-L GND #PWR074
+L GND #PWR075
 U 1 1 59EFDC50
 P 5400 1800
-F 0 "#PWR074" H 5400 1550 50  0001 C CNN
+F 0 "#PWR075" H 5400 1550 50  0001 C CNN
 F 1 "GND" H 5400 1650 50  0000 C CNN
 F 2 "" H 5400 1800 50  0001 C CNN

Commit message: Latest updates; preparing to move to github (I think).
git-svn-id: svn+ssh://dev.thehead.ca/depot/main/z80@636 995eaefb-0ce2-40e3-b8bc-69bf8729875b
Parts:
- removed unit 3 of U9
- added unit 3 of U4
Connections:
- net GND: now also U4.10, U4.7 (GND), U4.9
- net VCC: now also U4.14 (VCC)
Changed lines of the file:
@@
 $Descr A4 11693 8268
 encoding utf-8
-Sheet 7 8
+Sheet 7 9
 Title ""
-Date "2018-07-18"
-Rev "11"
+Date "2018-07-20"
+Rev "12"
 Comp ""
 Comment1 ""
@@
 $EndDescr
 $Comp
-L GND #PWR074
+L GND #PWR072
 U 1 1 59EFCC3B
 P 800 2350
-F 0 "#PWR074" H 800 2100 50  0001 C CNN
+F 0 "#PWR072" H 800 2100 50  0001 C CNN
 F 1 "GND" H 800 2200 50  0000 C CNN
 F 2 "" H 800 2350 50  0001 C CNN
@@
 	1    0    0    -1
 $EndComp
-$Comp
-L 74LS32 U4
-U 4 1 59EFD8A0
-P 3000 950
-F 0 "U4" H 3000 1000 50  0000 C CNN
-F 1 "74AHC32" H 3000 900 50  0000 C CNN
-F 2 "Housings_DIP:DIP-14_W7.62mm_LongPads" H 3000 950 50  0001 C CNN
-F 3 "" H 3000 950 50  0001 C CNN
-	4    3000 950
-	1    0    0    -1
-$EndComp
 NoConn ~ 4900 850
 NoConn ~ 4900 1250
-NoConn ~ 3600 950
 $Comp
-L GND #PWR075
-U 1 1 59EFDA1E
-P 2400 1350
-F 0 "#PWR075" H 2400 1100 50  0001 C CNN
-F 1 "GND" H 2400 1200 50  0000 C CNN
-F 2 "" H 2400 1350 50  0001 C CNN
-F 3 "" H 2400 1350 50  0001 C CNN
-	1    2400 1350
-	1    0    0    -1
-$EndComp
-$Comp
-L GND #PWR076
+L GND #PWR073
 U 1 1 59EFDA40
 P 4000 1600
-F 0 "#PWR076" H 4000 1350 50  0001 C CNN
+F 0 "#PWR073" H 4000 1350 50  0001 C CNN
 F 1 "GND" H 4000 1450 50  0000 C CNN
 F 2 "" H 4000 1600 50  0001 C CNN
@@
 	1    0    0    -1
 $EndComp
-Connection ~ 2400 1050
 Wire Wire Line
 	4000 850  4000 1600
 Connection ~ 4000 1250
-$Comp
-L 74HC02 U9
-U 3 1 59EFDB7C
-P 6000 950
-F 0 "U9" H 6000 1000 50  0000 C CNN
-F 1 "74AHC02" H 6050 900 50  0000 C CNN
-F 2 "Housings_DIP:DIP-14_W7.62mm_LongPads" H 6000 950 50  0001 C CNN
-F 3 "" H 6000 950 50  0001 C CNN
-	3    6000 950
-	1    0    0    -1
-$EndComp
 $Comp
 L 74HC02 U9
@@
 	1    0    0    -1
 $EndComp
-NoConn ~ 6600 950
 NoConn ~ 6600 1400
 $Comp
-L GND #PWR077
+L GND #PWR074
 U 1 1 59EFDC50
 P 5400 1800
-F 0 "#PWR077" H 5400 1550 50  0001 C CNN
+F 0 "#PWR074" H 5400 1550 50  0001 C CNN
 F 1 "GND" H 5400 1650 50  0000 C CNN
 F 2 "" H 5400 1800 50  0001 C CNN
@@
 	1    0    0    -1
 $EndComp
-Wire Wire Line
-	5400 850  5400 1800
-Connection ~ 5400 1050
-Connection ~ 5400 1300
 Connection ~ 5400 1500
 Wire Wire Line
-	2400 850  2400 1350
+	5400 1300 5400 1800
+$Comp
+L 74LS32 U4
+U 4 1 5B52E72D
+P 2950 1400
+F 0 "U4" H 2950 1450 50  0000 C CNN
+F 1 "74AHC32" H 2950 1350 50  0000 C CNN
+F 2 "Housings_DIP:DIP-14_W7.62mm_LongPads" H 2950 1400 50  0001 C CNN
+F 3 "" H 2950 1400 50  0001 C CNN
+	4    2950 1400
+	1    0    0    -1
+$EndComp
+$Comp
+L 74LS32 U4
+U 3 1 5B52E734
+P 2950 950
+F 0 "U4" H 2950 1000 50  0000 C CNN
+F 1 "74AHC32" H 2950 900 50  0000 C CNN
+F 2 "Housings_DIP:DIP-14_W7.62mm_LongPads" H 2950 950 50  0001 C CNN
+F 3 "" H 2950 950 50  0001 C CNN
+	3    2950 950
+	1    0    0    -1
+$EndComp
+NoConn ~ 3550 950
+NoConn ~ 3550 1400
+$Comp
+L GND #PWR075
+U 1 1 5B52E856
+P 2350 1850
+F 0 "#PWR075" H 2350 1600 50  0001 C CNN
+F 1 "GND" H 2350 1700 50  0000 C CNN
+F 2 "" H 2350 1850 50  0001 C CNN
+F 3 "" H 2350 1850 50  0001 C CNN
+	1    2350 1850
+	1    0    0    -1
+$EndComp
+Wire Wire Line
+	2350 850  2350 1850
+Connection ~ 2350 1050
+Connection ~ 2350 1300
+Connection ~ 2350 1500
 $EndSCHEMATC
