File: kicad/spares.sch (KiCad schematic (older format))
At the start: 4 parts, among them U16 74AHC08, U2 74AHC14, U4 74AHC32, U9 74AHC02

Commit message: Update to Kicad 5
Parts:
- U16: symbol 74LS08 -> 74xx:74LS08
- U2: symbol 74HC14 -> 74xx:74HC14
- U4: symbol 74LS32 -> 74xx:74LS32
- U9: symbol 74HC02 -> 74xx:74HC02
Connections:
- wire segments 4 -> 14
Other:
- moved on the sheet: U2C, U2D, U9D
