File: kicad/joystick.sch (KiCad schematic (older format))
At the start: 16 parts, among them U13 74AHC541, U14 74AHC541

Commit message: Assign footprints.
Parts:
- R10, R11, R2, R3, R4, R5, R6, R7, R8, R9: footprint Resistors_THT:R_Axial_DIN0204_L3.6mm_D1.6mm_P5.08mm_Horizontal -> Resistors_SMD:R_0805_HandSoldering
- U13, U14: footprint Housings_DIP:DIP-20_W7.62mm_LongPads -> Housings_SSOP:TSSOP-20_4.4x6.5mm_Pitch0.65mm
Changed lines of the file:
@@
 F 0 "U13" H 5050 3300 50  0000 C CNN
 F 1 "74AHC541" H 4650 2000 50  0000 C CNN
-F 2 "Housings_DIP:DIP-20_W7.62mm_LongPads" H 4850 2650 50  0001 C CNN
+F 2 "Housings_SSOP:TSSOP-20_4.4x6.5mm_Pitch0.65mm" H 4850 2650 50  0001 C CNN
 F 3 "" H 4850 2650 50  0001 C CNN
 	1    4850 2650
@@
 F 0 "R2" V 5530 1900 50  0000 C CNN
 F 1 "10K" V 5450 1900 50  0000 C CNN
-F 2 "Resistors_THT:R_Axial_DIN0204_L3.6mm_D1.6mm_P5.08mm_Horizontal" V 5380 1900 50  0001 C CNN
+F 2 "Resistors_SMD:R_0805_HandSoldering" V 5380 1900 50  0001 C CNN
 F 3 "" H 5450 1900 50  0001 C CNN
 	1    5450 1900
@@
 F 0 "R4" V 5730 1900 50  0000 C CNN
 F 1 "10K" V 5650 1900 50  0000 C CNN
-F 2 "Resistors_THT:R_Axial_DIN0204_L3.6mm_D1.6mm_P5.08mm_Horizontal" V 5580 1900 50  0001 C CNN
+F 2 "Resistors_SMD:R_0805_HandSoldering" V 5580 1900 50  0001 C CNN
 F 3 "" H 5650 1900 50  0001 C CNN
 	1    5650 1900
@@
 F 0 "R6" V 5930 1900 50  0000 C CNN
 F 1 "10K" V 5850 1900 50  0000 C CNN
-F 2 "Resistors_THT:R_Axial_DIN0204_L3.6mm_D1.6mm_P5.08mm_Horizontal" V 5780 1900 50  0001 C CNN
+F 2 "Resistors_SMD:R_0805_HandSoldering" V 5780 1900 50  0001 C CNN
 F 3 "" H 5850 1900 50  0001 C CNN
 	1    5850 1900
@@
 F 0 "R8" V 6130 1900 50  0000 C CNN
 F 1 "10K" V 6050 1900 50  0000 C CNN
-F 2 "Resistors_THT:R_Axial_DIN0204_L3.6mm_D1.6mm_P5.08mm_Horizontal" V 5980 1900 50  0001 C CNN
+F 2 "Resistors_SMD:R_0805_HandSoldering" V 5980 1900 50  0001 C CNN
 F 3 "" H 6050 1900 50  0001 C CNN
 	1    6050 1900
@@
 F 0 "R10" V 6330 1900 50  0000 C CNN
 F 1 "10K" V 6250 1900 50  0000 C CNN
-F 2 "Resistors_THT:R_Axial_DIN0204_L3.6mm_D1.6mm_P5.08mm_Horizontal" V 6180 1900 50  0001 C CNN
+F 2 "Resistors_SMD:R_0805_HandSoldering" V 6180 1900 50  0001 C CNN
 F 3 "" H 6250 1900 50  0001 C CNN
 	1    6250 1900
@@
 F 0 "U14" H 5050 5350 50  0000 C BNN
 F 1 "74AHC541" H 4650 4050 50  0000 C TNN
-F 2 "Housings_DIP:DIP-20_W7.62mm_LongPads" H 4850 4700 50  0001 C CNN
+F 2 "Housings_SSOP:TSSOP-20_4.4x6.5mm_Pitch0.65mm" H 4850 4700 50  0001 C CNN
 F 3 "" H 4850 4700 50  0001 C CNN
 	1    4850 4700
@@
 F 0 "R3" V 5530 3950 50  0000 C CNN
 F 1 "10K" V 5450 3950 50  0000 C CNN
-F 2 "Resistors_THT:R_Axial_DIN0204_L3.6mm_D1.6mm_P5.08mm_Horizontal" V 5380 3950 50  0001 C CNN
+F 2 "Resistors_SMD:R_0805_HandSoldering" V 5380 3950 50  0001 C CNN
 F 3 "" H 5450 3950 50  0001 C CNN
 	1    5450 3950
@@
 F 0 "R5" V 5730 3950 50  0000 C CNN
 F 1 "10K" V 5650 3950 50  0000 C CNN
-F 2 "Resistors_THT:R_Axial_DIN0204_L3.6mm_D1.6mm_P5.08mm_Horizontal" V 5580 3950 50  0001 C CNN
+F 2 "Resistors_SMD:R_0805_HandSoldering" V 5580 3950 50  0001 C CNN
 F 3 "" H 5650 3950 50  0001 C CNN
 	1    5650 3950
@@
 F 0 "R7" V 5930 3950 50  0000 C CNN
 F 1 "10K" V 5850 3950 50  0000 C CNN
-F 2 "Resistors_THT:R_Axial_DIN0204_L3.6mm_D1.6mm_P5.08mm_Horizontal" V 5780 3950 50  0001 C CNN
+F 2 "Resistors_SMD:R_0805_HandSoldering" V 5780 3950 50  0001 C CNN
 F 3 "" H 5850 3950 50  0001 C CNN
 	1    5850 3950
@@
 F 0 "R9" V 6130 3950 50  0000 C CNN
 F 1 "10K" V 6050 3950 50  0000 C CNN
-F 2 "Resistors_THT:R_Axial_DIN0204_L3.6mm_D1.6mm_P5.08mm_Horizontal" V 5980 3950 50  0001 C CNN
+F 2 "Resistors_SMD:R_0805_HandSoldering" V 5980 3950 50  0001 C CNN
 F 3 "" H 6050 3950 50  0001 C CNN
 	1    6050 3950
@@
 F 0 "R11" V 6330 3950 50  0000 C CNN
 F 1 "10K" V 6250 3950 50  0000 C CNN
-F 2 "Resistors_THT:R_Axial_DIN0204_L3.6mm_D1.6mm_P5.08mm_Horizontal" V 6180 3950 50  0001 C CNN
+F 2 "Resistors_SMD:R_0805_HandSoldering" V 6180 3950 50  0001 C CNN
 F 3 "" H 6250 3950 50  0001 C CNN
 	1    6250 3950

Commit message: First pass layout of revised board complete.
Connections:
- net GND: now also U13.7 (A5), U13.8 (A6); no longer U14.7 (A5), U14.8 (A6)
- net ~SDCD: now also U14.8 (A6); no longer U13.8 (A6)
- net ~SDWP: now also U14.7 (A5); no longer U13.7 (A5)
Changed lines of the file:
@@
 Sheet 2 11
 Title "Joystick Ports"
-Date "2019-04-11"
+Date "2019-04-15"
 Rev "1"
 Comp ""
@@
 L power:GND #PWR028
 U 1 1 59D6AB9F
-P 5500 4700
-F 0 "#PWR028" H 5500 4450 50  0001 C CNN
-F 1 "GND" H 5500 4550 50  0000 C CNN
-F 2 "" H 5500 4700 50  0001 C CNN
-F 3 "" H 5500 4700 50  0001 C CNN
-	1    5500 4700
-	1    0    0    -1
-$EndComp
-Wire Wire Line
-	5350 4700 5500 4700
+P 5350 4900
+F 0 "#PWR028" H 5350 4650 50  0001 C CNN
+F 1 "GND" H 5350 4750 50  0000 C CNN
+F 2 "" H 5350 4900 50  0001 C CNN
+F 3 "" H 5350 4900 50  0001 C CNN
+	1    5350 4900
+	1    0    0    -1
+$EndComp
 Wire Wire Line
 	6750 4850 6500 4850
@@
 Wire Wire Line
 	2850 5900 5750 5900
-Text HLabel 2850 6000 0    60   Input ~ 0
+Text HLabel 2850 6250 0    60   Input ~ 0
 ~IORQ0
 Text HLabel 2850 5800 0    60   Input ~ 0
@@
 	5400 7550 5700 7550
 Wire Wire Line
-	5350 4900 5350 4800
-Wire Wire Line
-	5350 4800 5350 4700
-Connection ~ 5350 4800
-Connection ~ 5350 4700
-Wire Wire Line
 	3800 2150 4350 2150
 Wire Wire Line
@@
 	5400 2850 5350 2850
 Wire Wire Line
-	2850 6000 7400 6000
+	2850 6250 7400 6250
 Wire Wire Line
 	5350 3150 5350 3550
@@
 	5350 3550 7400 3550
 Wire Wire Line
-	7400 3550 7400 6000
-Wire Wire Line
-	5350 2750 5800 2750
-Wire Wire Line
-	5800 2750 5800 3450
-Wire Wire Line
-	5800 3450 7500 3450
-Wire Wire Line
-	7500 3450 7500 6100
-Wire Wire Line
-	7500 6100 2850 6100
-Wire Wire Line
-	5350 2650 5900 2650
-Wire Wire Line
-	5900 2650 5900 3350
-Wire Wire Line
-	5900 3350 7600 3350
-Wire Wire Line
-	7600 3350 7600 6200
-Wire Wire Line
-	7600 6200 2850 6200
+	7400 3550 7400 6250
+Wire Wire Line
+	5850 6000 2850 6000
+Wire Wire Line
+	5950 6100 2850 6100
+Text HLabel 2850 6000 0    60   Input ~ 0
+~SDCD
 Text HLabel 2850 6100 0    60   Input ~ 0
-~SDCD
-Text HLabel 2850 6200 0    60   Input ~ 0
 ~SDWP
+Wire Wire Line
+	5350 2650 5350 2750
+Wire Wire Line
+	5350 2750 5350 2850
+Connection ~ 5350 2750
+Connection ~ 5350 2850
+Wire Wire Line
+	5850 6000 5850 4800
+Wire Wire Line
+	5850 4800 5350 4800
+Wire Wire Line
+	5950 6100 5950 4700
+Wire Wire Line
+	5950 4700 5350 4700
 Wire Bus Line
 	3700 2250 3700 5100
