File: kicad/joystick.sch (KiCad schematic (older format))
At the start: 16 parts, among them U13 74AHC541, U14 74AHC541

Commit message: Fix schematic so that ~SDWP signal is named SDWP instead, as it is active high, not active low. There is no change to connectivity, this is only a descriptive fix.
Connections:
- net ~SDWP renamed SDWP
Changed lines of the file:
@@
 Sheet 2 11
 Title "Joystick Ports"
-Date "2019-04-15"
+Date "2019-06-02"
 Rev "1"
 Comp ""
@@
 ~SDCD
 Text HLabel 2850 6100 0    60   Input ~ 0
-~SDWP
+SDWP
 Wire Wire Line
 	5350 2650 5350 2750
