File: kicad/zed-80.kicad_pcb (KiCad board)
At the start: 2 copper layers, 145 x 169 mm, 97 parts, among them J1 Conn_02x08_Odd_Even, J2 KMDGX-6S-BS, J3 Conn_02x20_Odd_Even, J5 USB_B, J6 PWR, SW1 KS01Q, U1 Z80CPU, U10 Z84C40, U11 SP232E, U12 SP232E, U13 74AHC541, U14 74AHC541, U15 Z84C20, U16 74AHC08, U17 Z84C30, U18 74HC164, U19 74HC164, U2 74AHC14, U3 SST39SF010, U4 74AHC32, U5 AS6C1008-55PCN, U6 74AHC138, U7 74AC574, U8 74AC574, U9 74AHC02, X1 ACH10MHZ, X2 1.8432MHz

Commit message: First pass layout of revised board complete.
Parts:
- removed C24: 10uF, Capacitors_THT:CP_Radial_D5.0mm_P2.50mm
- removed J1: Conn_02x08_Odd_Even, Pin_Headers:Pin_Header_Straight_2x08_Pitch2.54mm
- removed REF** (x4): MountingHole_3.2mm_M3_Pad, Mounting_Holes:MountingHole_3.2mm_M3_Pad
- added C30: 4.7uF, Capacitors_SMD:C_0805_HandSoldering, F.Cu at (22.9, 45.5)
- added C31: 0.1uF, Capacitors_THT:C_Disc_D4.3mm_W1.9mm_P5.00mm, F.Cu at (68.8, 147.1)
- added C32: 0.1uF, Capacitors_THT:C_Disc_D4.3mm_W1.9mm_P5.00mm, F.Cu at (71.5, 152.1)
- added C33: 0.1uF, Capacitors_THT:C_Disc_D4.3mm_W1.9mm_P5.00mm, F.Cu at (87.2, 160.2)
- added C34: 10uF, Capacitors_THT:CP_Radial_D5.0mm_P2.50mm, F.Cu at (87.6, 162.9)
- added C35: 0.1uF, Capacitors_THT:C_Disc_D4.3mm_W1.9mm_P5.00mm, F.Cu at (86.2, 152.5)
- added C36: 0.1uF, Capacitors_THT:C_Disc_D4.3mm_W1.9mm_P5.00mm, F.Cu at (128.1, 147.2)
- added C37: 0.1uF, Capacitors_THT:C_Disc_D4.3mm_W1.9mm_P5.00mm, F.Cu at (47.6, 149.9)
- added C38: 0.1uF, Capacitors_THT:C_Disc_D4.3mm_W1.9mm_P5.00mm, F.Cu at (77.6, 144.3)
- added C39: 0.1uF, Capacitors_THT:C_Disc_D4.3mm_W1.9mm_P5.00mm, F.Cu at (118.6, 135.2)
- added C40: 0.1uF, Capacitors_THT:C_Disc_D4.3mm_W1.9mm_P5.00mm, F.Cu at (127.8, 134.3)
- added C41: 0.1uF, Capacitors_THT:C_Disc_D4.3mm_W1.9mm_P5.00mm, F.Cu at (19.1, 80.0)
- added C42: 0.1uF, Capacitors_THT:C_Disc_D4.3mm_W1.9mm_P5.00mm, F.Cu at (138.8, 81.5)
- added C43: 0.1uF, Capacitors_THT:C_Disc_D4.3mm_W1.9mm_P5.00mm, F.Cu at (64.5, 51.0)
- added C44: 47uF, Capacitors_THT:CP_Radial_D6.3mm_P2.50mm, F.Cu at (126.5, 36.3)
- added C45: 4.7uF, Capacitors_SMD:C_0805_HandSoldering, F.Cu at (18.3, 45.5)
- added D2: D_ALT, Diodes_SMD:D_SOT-23_ANK, F.Cu at (55.8, 149.7)
- added D3: D_ALT, Diodes_SMD:D_SOT-23_ANK, F.Cu at (52.3, 146.2)
- added D4: D_ALT, Diodes_SMD:D_SOT-23_ANK, F.Cu at (53.9, 142.6)
- added D5: D_ALT, Diodes_SMD:D_SOT-23_ANK, F.Cu at (52.4, 139.1)
- added H1: 3.2mm M3, Mounting_Holes:MountingHole_3.2mm_M3_Pad, F.Cu at (20.0, 20.0)
- added H2: 3.2mm M3, Mounting_Holes:MountingHole_3.2mm_M3_Pad, F.Cu at (155.0, 20.0)
- added H3: 3.2mm M3, Mounting_Holes:MountingHole_3.2mm_M3_Pad, F.Cu at (20.0, 179.0)
- added H4: 3.2mm M3, Mounting_Holes:MountingHole_3.2mm_M3_Pad, F.Cu at (155.0, 179.0)
- added J4: Conn_02x20_Odd_Even, Pin_Headers:Pin_Header_Straight_2x20_Pitch2.54mm, F.Cu at (84.0, 156.6)
- added J7: SD_Card, z80_footprints:101-00405, F.Cu at (133.0, 156.6)
- added J8: SJ1-3523N, z80_footprints:SJ1-3523N, F.Cu at (142.3, 23.3)
- added J9: Conn_02x09_Odd_Even, Pin_Headers:Pin_Header_Straight_2x09_Pitch2.54mm, F.Cu at (152.8, 27.8)
- added R32: 10K, Resistors_SMD:R_0805_HandSoldering, F.Cu at (74.0, 152.3)
- added R33: 50K, Resistors_SMD:R_0805_HandSoldering, F.Cu at (153.1, 163.2)
- added R34: 10K, Resistors_SMD:R_0805_HandSoldering, F.Cu at (153.1, 166.7)
- added R35: 10K, Resistors_SMD:R_0805_HandSoldering, F.Cu at (153.1, 159.8)
- added R36: 100R, Resistors_SMD:R_0805_HandSoldering, F.Cu at (121.6, 34.1)
- added R37: 1K, Resistors_SMD:R_0805_HandSoldering, F.Cu at (132.8, 26.3)
- added R38: 1K, Resistors_SMD:R_0805_HandSoldering, F.Cu at (132.8, 22.4)
- added R39: 1K, Resistors_SMD:R_0805_HandSoldering, F.Cu at (132.8, 18.7)
- added U20: AP2114HA-33, TO_SOT_Packages_SMD:SOT-223-3_TabPin2, F.Cu at (20.6, 40.1)
- added U21: 74LVC4245A, Housings_SSOP:TSSOP-24_4.4x7.8mm_Pitch0.65mm, F.Cu at (63.2, 149.6)
- added U22: 74LVC244A, Housings_SSOP:TSSOP-20_4.4x6.5mm_Pitch0.65mm, F.Cu at (81.2, 150.0)
- added U23: 74AC273, Housings_SSOP:TSSOP-20_4.4x6.5mm_Pitch0.65mm, F.Cu at (75.1, 139.3)
- added U24: 74HC670, Housings_SOIC:SOIC-16_3.9x9.9mm_Pitch1.27mm, F.Cu at (45.1, 143.2)
- added U25: 74HCT164, Housings_SSOP:TSSOP-14_4.4x5mm_Pitch0.65mm, F.Cu at (116.1, 139.4)
- added U26: 74AHC541, Housings_SSOP:TSSOP-20_4.4x6.5mm_Pitch0.65mm, F.Cu at (125.2, 140.2)
- added U27: 74LV165, Housings_SSOP:TSSOP-16_4.4x5mm_Pitch0.65mm, F.Cu at (121.7, 149.6)
- added U28: 74HC390, Housings_SSOP:TSSOP-16_4.4x5mm_Pitch0.65mm, F.Cu at (24.6, 82.5)
- added U29: AY-3-8910, Housings_DIP:DIP-40_W15.24mm_Socket, F.Cu at (148.9, 78.5)
- added U30: 74AHC541, Housings_SSOP:TSSOP-20_4.4x6.5mm_Pitch0.65mm, F.Cu at (62.0, 56.0)
- R10, R11, R18, R2, R29, R3, R30, R31, R4, R5, R6, R7, R8, R9: footprint Resistors_THT:R_Axial_DIN0204_L3.6mm_D1.6mm_P5.08mm_Horizontal -> Resistors_SMD:R_0805_HandSoldering
- U1, U10, U15: footprint Housings_DIP:DIP-40_W15.24mm_Socket_LongPads -> Housings_DIP:DIP-40_W15.24mm_Socket
- U11, U12: footprint Housings_DIP:DIP-16_W7.62mm_LongPads -> Housings_DIP:DIP-16_W7.62mm
- U13, U14: footprint Housings_DIP:DIP-20_W7.62mm_LongPads -> Housings_SSOP:TSSOP-20_4.4x6.5mm_Pitch0.65mm
- U16, U2, U4, U9: footprint Housings_DIP:DIP-14_W7.62mm_LongPads -> Housings_DIP:DIP-14_W7.62mm
- U18, U19: value 74HC164 -> 74HCT164; footprint Housings_DIP:DIP-14_W7.62mm_LongPads -> Housings_SSOP:TSSOP-14_4.4x5mm_Pitch0.65mm
- U3, U5: footprint Housings_DIP:DIP-32_W15.24mm_Socket_LongPads -> Housings_DIP:DIP-32_W15.24mm_Socket
- U6: value 74AHC138 -> 74HC154; footprint Housings_DIP:DIP-16_W7.62mm_LongPads -> Housings_SOIC:SOIC-24W_7.5x15.4mm_Pitch1.27mm
- U7, U8: value 74AC574 -> 74AC273; footprint Housings_DIP:DIP-20_W7.62mm_LongPads -> Housings_SSOP:TSSOP-20_4.4x6.5mm_Pitch0.65mm
- X1: value ACH10MHZ -> ACH20MHZ
- moved X2 122.4 mm to (19.2, 52.6)
- moved C27 101.9 mm to (44.8, 58.9)
- moved U17 101.7 mm to (43.6, 66.2)
- moved X1 93.8 mm to (19.2, 67.8), turned to 270 degrees
- moved C20 76.7 mm to (156.3, 85.5), turned to 270 degrees
- moved U9 59.1 mm to (138.1, 91.6), turned to 90 degrees
- moved C29 55.1 mm to (58.0, 32.2)
- moved C28 50.1 mm to (58.0, 40.6)
- moved R11 45.5 mm to (69.3, 165.0), turned to 270 degrees
- moved R3 44.4 mm to (72.0, 165.0), turned to 270 degrees
- moved R5 41.2 mm to (74.6, 165.0), turned to 270 degrees
- moved R7 38.1 mm to (77.3, 165.0), turned to 270 degrees
- moved R9 35.1 mm to (79.9, 165.0), turned to 270 degrees
- moved U19 33.1 mm to (55.5, 36.4)
- moved U18 32.6 mm to (55.5, 44.8)
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Connections:
- J3 pad 28: /~IORQ7 -> /~IORQ15
- J3 pad 30: /~IORQ5 -> /~IORQ14
- J3 pad 32: /~IORQ6 -> /~IORQ13
- U10 pad 16: (no net) -> /LCD/BL
- U14 pad 7: GND -> /Joystick Ports/~SDWP
- U14 pad 8: GND -> /Joystick Ports/~SDCD
- U15 pad 27: /PIO/SR0 -> /Audio/D0
- U15 pad 28: /PIO/SR1 -> /Audio/D1
- U15 pad 29: /PIO/SR2 -> /Audio/D2
- U15 pad 30: /PIO/SR3 -> /Audio/D3
- U15 pad 31: /PIO/SR4 -> /Audio/D4
- U15 pad 32: /PIO/SR5 -> /Audio/D5
- U15 pad 33: /PIO/SR6 -> /Audio/D6
- U15 pad 34: /PIO/SR7 -> /Audio/D7
- U15 pad 7: Net-(J1-Pad15) -> /PIO/PIOA7
- U15 pad 8: Net-(J1-Pad13) -> /LCD/INT
- U18 pad 2: /PIO/~KDAT -> VCC
- U19 pad 2: /PIO/SR2 -> VCC
- U2 pad 5: GND -> /MMUEN
- U2 pad 6: (no net) -> Net-(U2-Pad6)
- U3 pad 2: GND -> /PA16
- U3 pad 29: /A14 -> /PA14
- U3 pad 3: /A15 -> /PA15
- U4 pad 1: Net-(U4-Pad1) -> /~IORQ6
- U4 pad 10: /A14 -> /~IORQ8
- U4 pad 2: /A15 -> /~WR
- U4 pad 3: Net-(U4-Pad3) -> Net-(U24-Pad12)
- U4 pad 5: Net-(U4-Pad3) -> /PA17
- U4 pad 8: Net-(U4-Pad1) -> Net-(U27-Pad1)
- U4 pad 9: /A13 -> /~WR
- U5 pad 2: GND -> /PA16
- U5 pad 3: /A14 -> /PA14
- U5 pad 30: Net-(U4-Pad3) -> /PA17
- U5 pad 31: /A15 -> /PA15
- U6 pad 1: /A4 -> /~IORQ0
- U6 pad 10: /~IORQ5 -> /~IORQ9
- U6 pad 11: /~IORQ4 -> (no net)
- U6 pad 12: /~IORQ3 -> GND
- U6 pad 13: /~IORQ2 -> (no net)
- U6 pad 14: /~IORQ1 -> (no net)
- U6 pad 15: /~IORQ0 -> /~IORQ13
- U6 pad 16: VCC -> /~IORQ14
- U6 pad 2: /A5 -> /~IORQ1
- U6 pad 3: /A6 -> /~IORQ2
- U6 pad 4: /~IORQ -> /~IORQ3
- U6 pad 5: /A7 -> /~IORQ4
- U6 pad 6: VCC -> /~IORQ5
- U6 pad 7: /~IORQ7 -> /~IORQ6
- U6 pad 8: GND -> /~IORQ7
- U6 pad 9: /~IORQ6 -> /~IORQ8
- U7 pad 1: GND -> /~RESET
- U7 pad 12: Net-(R20-Pad2) -> Net-(R16-Pad2)
- U7 pad 13: Net-(R19-Pad2) -> /D4
- U7 pad 14: Net-(R17-Pad2) -> /D5
- U7 pad 15: Net-(R16-Pad2) -> Net-(R17-Pad2)
- U7 pad 16: Net-(R15-Pad2) -> Net-(R19-Pad2)
- U7 pad 17: Net-(R14-Pad2) -> /D6
- U7 pad 18: Net-(R13-Pad2) -> /D7
- U7 pad 19: Net-(R12-Pad2) -> Net-(R20-Pad2)
- U7 pad 2: /D0 -> Net-(R12-Pad2)
- U7 pad 3: /D1 -> /D0
- U7 pad 4: /D2 -> /D1
- U7 pad 5: /D3 -> Net-(R13-Pad2)
- U7 pad 6: /D4 -> Net-(R14-Pad2)
- U7 pad 7: /D5 -> /D2
- U7 pad 8: /D6 -> /D3
- U7 pad 9: /D7 -> Net-(R15-Pad2)
- U8 pad 1: GND -> /~RESET
- U8 pad 12: Net-(R28-Pad2) -> Net-(R25-Pad2)
- U8 pad 13: Net-(R27-Pad2) -> /D4
- U8 pad 14: Net-(R26-Pad2) -> /D5
- U8 pad 15: Net-(R25-Pad2) -> Net-(R26-Pad2)
- U8 pad 16: Net-(R24-Pad2) -> Net-(R27-Pad2)
- U8 pad 17: Net-(R23-Pad2) -> /D6
- U8 pad 18: Net-(R22-Pad2) -> /D7
- U8 pad 19: Net-(R21-Pad2) -> Net-(R28-Pad2)
- U8 pad 2: /D0 -> Net-(R21-Pad2)
- U8 pad 3: /D1 -> /D0
- U8 pad 4: /D2 -> /D1
- U8 pad 5: /D3 -> Net-(R22-Pad2)
- U8 pad 6: /D4 -> Net-(R23-Pad2)
- U8 pad 7: /D5 -> /D2
- U8 pad 8: /D6 -> /D3
- U8 pad 9: /D7 -> Net-(R24-Pad2)
- U9 pad 10: (no net) -> Net-(U23-Pad11)
- U9 pad 8: GND -> /~WR
- U9 pad 9: GND -> /~IORQ7
- X1 pad 5: /CLK -> Net-(U28-Pad1)
Routing:
- net +3V3: track 0.00 -> 291.0 mm, vias 0 -> 2
- net VCC: track 594.7 -> 782.0 mm, vias 6 -> 17
- net /~WR: track 136.0 -> 307.1 mm, vias 3 -> 4
- net /LCD/BL: track 0.00 -> 160.6 mm, vias 0 -> 3
- net /CLK2M: track 0.00 -> 155.0 mm, vias 0 -> 1
- net /~IORQ0: track 106.9 -> 256.6 mm, vias 0 -> 2
- net /MMUEN: track 0.00 -> 148.8 mm, vias 0 -> 4
- net /BDIR: track 0.00 -> 144.4 mm, vias 0 -> 2
- net Net-(U23-Pad11): track 0.00 -> 142.8 mm, vias 0 -> 1
- net /~IORQ8: track 0.00 -> 139.7 mm, vias 0 -> 3
- net /BC1: track 0.00 -> 138.7 mm, vias 0 -> 2
- net /~IORQ7: track 11.0 -> 146.6 mm, vias 0 -> 1
- net GND: track 619.0 -> 750.1 mm, vias 3 -> 16
- net /~IORQ9: track 0.00 -> 125.7 mm, vias 0 -> 4
- net Net-(U2-Pad6): track 0.00 -> 110.0 mm, vias 0 -> 1
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Other:
- net class Default: clearance 0.2032 -> 0.1524; trace_width 0.2032 -> 0.1524
- rule trace_clearance: 0.2032 -> 0.1524
- board text removed: "Z80 Prototype rev 10 2018/06/12 dan.collens@gmail.com"

Commit message: Finalize layout of ZED-80 rev. 1
Parts:
- moved J8 1.20 mm to (142.3, 24.5)
Routing:
- net GND: track 750.1 -> 776.3 mm, vias 16 -> 17
- net Net-(C44-Pad2): track 40.1 -> 41.3 mm
Other:
- outline, holes or cut-outs redrawn
- board text added: "ZED-80 rev. 1 2019/04/15 dan.collens@gmail.com"
Changed lines of the file:
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@@
   (general
     (thickness 1.6002)
-    (drawings 4)
-    (tracks 4794)
+    (drawings 9)
+    (tracks 4801)
     (zones 0)
     (modules 138)
@@
   (page USLetter)
   (title_block
-    (title "Z80 Prototype")
-    (date 2018-06-12)
-    (rev 10)
+    (title "ZED-80 Personal Computer")
+    (date 2019-04-15)
+    (rev 1)
   )
   (layers
@@
   )
   (setup
-    (last_trace_width 0.508)
+    (last_trace_width 0.1524)
     (user_trace_width 0.1524)
     (user_trace_width 0.254)
@@
   )
   (module z80_footprints:SJ1-3523N (layer F.Cu)
-    (at 142.35 23.3)
+    (at 142.3 24.5)
     (descr "CUI 3.5mm stereo mini jack, no switch")
-    (fp_text reference J8 (at 0 4.2) (layer F.SilkS)
+    (fp_text reference J8 (at 7.4 -2.25) (layer F.SilkS)
       (effects (font (size 1 1) (thickness 0.15)))
     )
@@
       (net 13 GND))
   )
+  (gr_text "ZED-80 rev. 1\n2019/04/15\ndan.collens@gmail.com" (at 94.95 179.5) (layer F.SilkS)
+    (effects (font (size 1.2 1.2) (thickness 0.18)) (justify left))
+  )
+  (gr_line (start 140.25 16.3) (end 140.25 15) (layer Edge.Cuts) (width 0.15))
+  (gr_line (start 144.35 16.3) (end 140.25 16.3) (layer Edge.Cuts) (width 0.15))
+  (gr_line (start 144.35 15) (end 144.35 16.3) (layer Edge.Cuts) (width 0.15))
+  (gr_line (start 160 15) (end 144.35 15) (layer Edge.Cuts) (width 0.15))
   (gr_line (start 15 184) (end 15 15) (layer Edge.Cuts) (width 0.15))
   (gr_line (start 160 184) (end 15 184) (layer Edge.Cuts) (width 0.15))
   (gr_line (start 160 15) (end 160 184) (layer Edge.Cuts) (width 0.15))
-  (gr_line (start 15 15) (end 160 15) (layer Edge.Cuts) (width 0.15))
+  (gr_line (start 15 15) (end 140.25 15) (layer Edge.Cuts) (width 0.15))
   (segment (start 133.35 139.4192) (end 133.35 142.01) (width 0.2032) (layer F.Cu) (net 1))
   (segment (start 133.35 138.2) (end 133.35 139.4192) (width 0.2032) (layer F.Cu) (net 1))
@@
   (segment (start 53 40.033) (end 51.317 38.35) (width 0.508) (layer B.Cu) (net 13))
   (segment (start 53 40.6) (end 53 40.033) (width 0.508) (layer B.Cu) (net 13))
+  (via (at 122.95 32.75) (size 0.6) (drill 0.3) (layers F.Cu B.Cu) (net 13))
+  (segment (start 122.95 32.75) (end 121.6 32.75) (width 0.1524) (layer F.Cu) (net 13))
+  (segment (start 138.5 19.5) (end 125.25 32.75) (width 0.1524) (layer B.Cu) (net 13))
+  (segment (start 125.25 32.75) (end 122.95 32.75) (width 0.1524) (layer B.Cu) (net 13))
+  (segment (start 142.3 19.5) (end 138.5 19.5) (width 0.1524) (layer B.Cu) (net 13))
   (segment (start 148.59 122.96) (end 148.59 121.52316) (width 0.2032) (layer F.Cu) (net 14))
   (segment (start 148.59 121.52316) (end 148.59 119.15) (width 0.2032) (layer F.Cu) (net 14))
@@
   (segment (start 61.3 89.6) (end 59.69 91.21) (width 0.508) (layer F.Cu) (net 19))
   (segment (start 62.6 89.6) (end 61.3 89.6) (width 0.508) (layer F.Cu) (net 19))
-  (segment (start 152.85 27.75) (end 143.6 27.75) (width 0.508) (layer F.Cu) (net 19))
   (via (at 139.9 31.45) (size 0.6) (drill 0.3) (layers F.Cu B.Cu) (net 19))
-  (segment (start 143.6 27.75) (end 139.9 31.45) (width 0.508) (layer F.Cu) (net 19))
   (segment (start 139.9 34.21) (end 133.71 40.4) (width 0.508) (layer B.Cu) (net 19))
   (segment (start 139.9 31.45) (end 139.9 34.21) (width 0.508) (layer B.Cu) (net 19))
@@
   (segment (start 59.01459 104.98541) (end 59.01459 149.43541) (width 0.508) (layer F.Cu) (net 19))
   (segment (start 64.77 95.02) (end 65.976401 96.226401) (width 0.508) (layer F.Cu) (net 19))
+  (segment (start 143.25 28.1) (end 139.9 31.45) (width 0.508) (layer F.Cu) (net 19))
+  (segment (start 152.5 28.1) (end 143.25 28.1) (width 0.508) (layer F.Cu) (net 19))
+  (segment (start 152.85 27.75) (end 152.5 28.1) (width 0.508) (layer F.Cu) (net 19))
   (segment (start 69.85 44.474) (end 69.85 45.8772) (width 0.2032) (layer F.Cu) (net 20))
   (segment (start 69.85 45.8772) (end 69.85 48.284) (width 0.2032) (layer F.Cu) (net 20))
@@
   (segment (start 131.4 30.4976) (end 126.55 35.3476) (width 0.1524) (layer F.Cu) (net 142))
   (segment (start 131.4 26.3) (end 131.4 30.4976) (width 0.1524) (layer F.Cu) (net 142))
-  (segment (start 137.35 22.1476) (end 137.35 23.3) (width 0.1524) (layer F.Cu) (net 143))
-  (segment (start 137.35 20.138518) (end 137.35 22.1476) (width 0.1524) (layer F.Cu) (net 143))
-  (segment (start 135.032881 17.821399) (end 137.35 20.138518) (width 0.1524) (layer F.Cu) (net 143))
   (segment (start 130.467119 17.821399) (end 135.032881 17.821399) (width 0.1524) (layer F.Cu) (net 143))
   (segment (start 130.421399 17.867119) (end 130.467119 17.821399) (width 0.1524) (layer F.Cu) (net 143))
   (segment (start 130.421399 29.928601) (end 130.421399 17.867119) (width 0.1524) (layer F.Cu) (net 143))
   (segment (start 126.55 33.8) (end 130.421399 29.928601) (width 0.1524) (layer F.Cu) (net 143))
-  (segment (start 147.35 22.9) (end 147.35 23.3) (width 0.1524) (layer F.Cu) (net 143))
-  (segment (start 138.178601 22.071399) (end 146.521399 22.071399) (width 0.1524) (layer F.Cu) (net 143))
-  (segment (start 137.35 22.9) (end 138.178601 22.071399) (width 0.1524) (layer F.Cu) (net 143))
-  (segment (start 146.521399 22.071399) (end 147.35 22.9) (width 0.1524) (layer F.Cu) (net 143))
-  (segment (start 137.35 23.3) (end 137.35 22.9) (width 0.1524) (layer F.Cu) (net 143))
+  (segment (start 137.3 23.3476) (end 137.3 24.5) (width 0.1524) (layer F.Cu) (net 143))
+  (segment (start 135.078601 21.126201) (end 137.3 23.3476) (width 0.1524) (layer F.Cu) (net 143))
+  (segment (start 135.078601 17.867119) (end 135.078601 21.126201) (width 0.1524) (layer F.Cu) (net 143))
+  (segment (start 135.032881 17.821399) (end 135.078601 17.867119) (width 0.1524) (layer F.Cu) (net 143))
+  (segment (start 147.3 24.1) (end 147.3 24.5) (width 0.1524) (layer F.Cu) (net 143))
+  (segment (start 138.128601 23.271399) (end 146.471399 23.271399) (width 0.1524) (layer F.Cu) (net 143))
+  (segment (start 137.3 24.1) (end 138.128601 23.271399) (width 0.1524) (layer F.Cu) (net 143))
+  (segment (start 146.471399 23.271399) (end 147.3 24.1) (width 0.1524) (layer F.Cu) (net 143))
+  (segment (start 137.3 24.5) (end 137.3 24.1) (width 0.1524) (layer F.Cu) (net 143))
   (via (at 41.05 145.15) (size 0.6) (drill 0.3) (layers F.Cu B.Cu) (net 144))
   (segment (start 42.395 145.15) (end 42.4 145.155) (width 0.1524) (layer F.Cu) (net 144))
@@
     (polygon
       (pts
-        (xy 15.6464 15.5688) (xy 159.512 15.5688) (xy 159.512 183.412) (xy 15.6464 183.412)
+        (xy 15.6464 15.5688) (xy 135.9 15.55) (xy 135.9 27.6) (xy 148.7 27.6) (xy 148.7 15.55)
+        (xy 159.512 15.5688) (xy 159.512 183.412) (xy 15.6464 183.412)
       )
     )
@@
     (polygon
       (pts
-        (xy 15.6464 15.5688) (xy 159.512 15.5688) (xy 159.512 183.412) (xy 15.6464 183.412)
+        (xy 15.6464 15.5688) (xy 135.9 15.55) (xy 135.9 18.1) (xy 148.7 18.1) (xy 148.7 15.5688)
+        (xy 159.512 15.5688) (xy 159.512 183.412) (xy 15.6464 183.412)
       )
     )
