File: kicad/CTC.sch (KiCad schematic (older format))
At the start: 3 parts, among them U17 Z84C30, X2 1.8432MHz

Commit message: Update to Kicad 5
Parts:
- C27: symbol C -> Device:C
- U17: symbol Z84C30 -> headquarters:Z84C30
- X2: symbol CXO_DIP8 -> Oscillator:CXO_DIP8
Connections:
- wire segments 34 -> 36
Changed lines of the file:
@@
-EESchema Schematic File Version 2
-LIBS:power
-LIBS:device
-LIBS:transistors
-LIBS:conn
-LIBS:linear
-LIBS:regul
-LIBS:74xx
-LIBS:cmos4000
-LIBS:adc-dac
-LIBS:memory
-LIBS:xilinx
-LIBS:microcontrollers
-LIBS:dsp
-LIBS:microchip
-LIBS:analog_switches
-LIBS:motorola
-LIBS:texas
-LIBS:intel
-LIBS:audio
-LIBS:interface
-LIBS:digital-audio
-LIBS:philips
-LIBS:display
-LIBS:cypress
-LIBS:siliconi
-LIBS:opto
-LIBS:atmel
-LIBS:contrib
-LIBS:valves
-LIBS:Zilog
-LIBS:Oscillators
-LIBS:switches
-LIBS:headquarters
+EESchema Schematic File Version 4
 LIBS:z80-cache
-EELAYER 25 0
+EELAYER 26 0
 EELAYER END
 $Descr USLetter 11000 8500
@@
 $EndDescr
 $Comp
-L Z84C30 U17
+L headquarters:Z84C30 U17
 U 1 1 59D9201C
 P 3500 3150
@@
 $EndComp
 $Comp
-L VCC #PWR066
+L power:VCC #PWR066
 U 1 1 59D9205A
 P 3500 1950
@@
 $EndComp
 $Comp
-L GND #PWR067
+L power:GND #PWR067
 U 1 1 59D92070
 P 3500 4950
@@
 Text HLabel 1100 2000 0    60   BiDi ~ 0
 D[0..7]
-Wire Bus Line
-	2550 2850 2550 2000
 Wire Bus Line
 	2550 2000 1100 2000
@@
 	1100 4450 2800 4450
 $Comp
-L C C27
+L Device:C C27
 U 1 1 59D92B9B
 P 4800 6750
@@
 $EndComp
 $Comp
-L GND #PWR068
+L power:GND #PWR068
 U 1 1 59D92BA2
 P 4550 6900
@@
 $EndComp
 $Comp
-L VCC #PWR069
+L power:VCC #PWR069
 U 1 1 59D92BAF
 P 4550 6600
@@
 Text Notes 4750 6550 0    60   ~ 0
 Near\nU17
-Connection ~ 4800 6600
-Connection ~ 4800 6900
 Wire Wire Line
 	4550 6600 4800 6600
@@
 	4300 2500 4200 2500
 Wire Wire Line
-	4200 2250 5200 2250
+	4200 2250 4300 2250
 Connection ~ 4300 2500
 $Comp
-L CXO_DIP8 X2
+L Oscillator:CXO_DIP8 X2
 U 1 1 59DCF0C2
 P 5500 2250
@@
 $EndComp
 $Comp
-L GND #PWR070
+L power:GND #PWR070
 U 1 1 59DCF0C9
 P 5500 2550
@@
 $EndComp
 $Comp
-L VCC #PWR071
+L power:VCC #PWR071
 U 1 1 59DCF0CF
 P 5500 1950
@@
 	5800 1950 5800 2250
 Wire Wire Line
-	4300 2250 4300 2750
+	4300 2250 4300 2500
 Connection ~ 4300 2250
 Text HLabel 6300 3000 2    60   Output ~ 0
@@
 Wire Wire Line
 	4400 3100 6300 3100
+Wire Wire Line
+	4300 2500 4300 2750
+Wire Wire Line
+	4300 2250 5200 2250
+Wire Bus Line
+	2550 2000 2550 2850
 $EndSCHEMATC
