File: kicad/MMU.sch (KiCad schematic (older format))
At the start: 10 parts, among them U23 74VHC175, U24 74HC670, U4 74AHC32, U9 74AHC02

Commit message: Working on SD card interface, cleaning up.
Parts:
- removed C36: 0.1uF, Capacitors_THT:C_Disc_D4.3mm_W1.9mm_P5.00mm, symbol Device:C
- removed U23: 74VHC175, symbol 74xx:74LS175
- removed U9: 74AHC02, Housings_DIP:DIP-14_W7.62mm_LongPads, symbol 74xx:74HC02
- added U2: 74AHC14, Housings_DIP:DIP-14_W7.62mm_LongPads, symbol 74xx:74HC14
Connections:
- net labels added: MMUENA
- net labels removed: ~IORQCTL, ~RESET
- wire segments 47 -> 31
- no-connect marks 6 -> 0
Other:
- note removed: "Near\nU23"
Changed lines of the file:
@@
 $Descr USLetter 11000 8500
 encoding utf-8
-Sheet 9 9
-Title ""
+Sheet 10 10
+Title "Memory Management Unit"
 Date "2018-07-20"
 Rev "12"
@@
 Text HLabel 2350 1850 0    60   Input ~ 0
 D[0..3]
-Text Label 4450 3700 0    60   ~ 0
-D0
-Text Label 4450 3900 0    60   ~ 0
-D1
-Text Label 4450 4100 0    60   ~ 0
-D2
-Text Label 4450 4300 0    60   ~ 0
-D3
-Entry Wire Line
-	4350 3600 4450 3700
-Entry Wire Line
-	4350 3800 4450 3900
-Entry Wire Line
-	4350 4000 4450 4100
-Entry Wire Line
-	4350 4200 4450 4300
 Text HLabel 2300 2400 0    60   Input ~ 0
 WA0
 Text HLabel 2300 2500 0    60   Input ~ 0
 WA1
-Text HLabel 2300 3650 0    60   Input ~ 0
+Text HLabel 2300 3300 0    60   Input ~ 0
 ~WR
 Text HLabel 2300 2750 0    60   Input ~ 0
@@
 Text Label 6150 2250 2    60   ~ 0
 A17
-Text HLabel 2300 4600 0    60   Input ~ 0
-~RESET
-NoConn ~ 6000 3900
-NoConn ~ 6000 4000
-NoConn ~ 6000 4100
-NoConn ~ 6000 4200
-NoConn ~ 6000 4300
-NoConn ~ 6000 4400
 $Comp
 L Device:D_ALT D2
@@
 Connection ~ 6550 3300
 Wire Wire Line
-	6250 3300 6250 3700
-Connection ~ 6250 3300
-Wire Wire Line
 	6250 2250 6250 3000
 Wire Wire Line
@@
 Wire Wire Line
 	7150 1950 7150 3000
-$Comp
-L 74xx:74LS175 U23
-U 1 1 5B5115BC
-P 5500 4100
-F 0 "U23" H 5500 4100 50  0000 C CNN
-F 1 "74VHC175" H 5600 3700 50  0000 C CNN
-F 2 "" H 5500 4100 50  0001 C CNN
-F 3 "" H 5500 4100 50  0001 C CNN
-	1    5500 4100
-	1    0    0    -1
-$EndComp
-Wire Wire Line
-	6250 3700 6000 3700
-Wire Wire Line
-	4950 3150 4950 2950
 Text HLabel 2300 3100 0    60   Input ~ 0
 ~IORQMMU
-Text HLabel 2300 4300 0    60   Input ~ 0
-~IORQCTL
 Wire Wire Line
 	4450 1950 4950 1950
@@
 Wire Wire Line
 	4700 2600 4950 2600
-Wire Wire Line
-	2300 3650 2650 3650
-Wire Wire Line
-	2650 3300 2650 3650
-$Comp
-L 74xx:74HC02 U9
-U 3 1 5B5124C8
-P 3250 4200
-AR Path="/5B5124C8" Ref="U9"  Part="3"
-AR Path="/5B502B1D/5B5124C8" Ref="U9"  Part="3"
-F 0 "U9" H 3250 4250 50  0000 C CNN
-F 1 "74AHC02" H 3300 4150 50  0000 C CNN
-F 2 "Housings_DIP:DIP-14_W7.62mm_LongPads" H 3250 4200 50  0001 C CNN
-F 3 "" H 3250 4200 50  0001 C CNN
-	3    3250 4200
-	1    0    0    -1
-$EndComp
-Connection ~ 2650 3650
-Wire Wire Line
-	3850 4200 3850 4500
-$Comp
-L Device:C C36
-U 1 1 5B522DC2
-P 4500 6400
-F 0 "C36" H 4525 6500 50  0000 L CNN
-F 1 "0.1uF" H 4525 6300 50  0000 L CNN
-F 2 "Capacitors_THT:C_Disc_D4.3mm_W1.9mm_P5.00mm" H 4538 6250 50  0001 C CNN
-F 3 "" H 4500 6400 50  0001 C CNN
-	1    4500 6400
-	1    0    0    -1
-$EndComp
 $Comp
 L power:GND #PWR094
 U 1 1 5B522DC9
-P 4250 6550
-F 0 "#PWR094" H 4250 6300 50  0001 C CNN
-F 1 "GND" H 4250 6400 50  0000 C CNN
-F 2 "" H 4250 6550 50  0001 C CNN
-F 3 "" H 4250 6550 50  0001 C CNN
-	1    4250 6550
+P 4550 6550
+F 0 "#PWR094" H 4550 6300 50  0001 C CNN
+F 1 "GND" H 4550 6400 50  0000 C CNN
+F 2 "" H 4550 6550 50  0001 C CNN
+F 3 "" H 4550 6550 50  0001 C CNN
+	1    4550 6550
 	1    0    0    -1
 $EndComp
@@
 L power:VCC #PWR095
 U 1 1 5B522DD6
-P 4250 6250
-F 0 "#PWR095" H 4250 6100 50  0001 C CNN
-F 1 "VCC" H 4250 6400 50  0000 C CNN
-F 2 "" H 4250 6250 50  0001 C CNN
-F 3 "" H 4250 6250 50  0001 C CNN
-	1    4250 6250
-	1    0    0    -1
-$EndComp
-Text Notes 4450 6200 0    60   ~ 0
-Near\nU23
+P 4550 6250
+F 0 "#PWR095" H 4550 6100 50  0001 C CNN
+F 1 "VCC" H 4550 6400 50  0000 C CNN
+F 2 "" H 4550 6250 50  0001 C CNN
+F 3 "" H 4550 6250 50  0001 C CNN
+	1    4550 6250
+	1    0    0    -1
+$EndComp
 Text Notes 4750 6200 0    60   ~ 0
 Near\nU24
-Connection ~ 4500 6250
-Connection ~ 4500 6550
-Wire Wire Line
-	4250 6550 4500 6550
-Wire Wire Line
-	4250 6250 4500 6250
 Wire Wire Line
 	6850 3300 7150 3300
@@
 	6550 3300 6850 3300
 Wire Wire Line
-	2650 3650 2650 4100
-Wire Wire Line
-	4500 6250 4800 6250
-Wire Wire Line
-	4500 6550 4800 6550
-Wire Wire Line
-	3550 4200 3850 4200
-Wire Wire Line
-	2950 4100 2650 4100
-Wire Wire Line
-	2300 4300 2950 4300
-Wire Wire Line
-	2300 4600 5000 4600
-Wire Wire Line
-	3850 4500 5000 4500
-Wire Wire Line
-	4450 4300 5000 4300
-Wire Wire Line
-	4450 4100 5000 4100
-Wire Wire Line
-	4450 3900 5000 3900
-Wire Wire Line
-	4450 3700 5000 3700
-$Comp
-L power:VCC #PWR0110
-U 1 1 5C333009
-P 5500 3400
-F 0 "#PWR0110" H 5500 3250 50  0001 C CNN
-F 1 "VCC" H 5517 3573 50  0000 C CNN
-F 2 "" H 5500 3400 50  0001 C CNN
-F 3 "" H 5500 3400 50  0001 C CNN
-	1    5500 3400
-	1    0    0    -1
-$EndComp
-$Comp
-L power:GND #PWR0111
-U 1 1 5C333057
-P 5500 4900
-F 0 "#PWR0111" H 5500 4650 50  0001 C CNN
-F 1 "GND" H 5505 4727 50  0000 C CNN
-F 2 "" H 5500 4900 50  0001 C CNN
-F 3 "" H 5500 4900 50  0001 C CNN
-	1    5500 4900
-	1    0    0    -1
-$EndComp
-Wire Wire Line
-	6000 3800 6050 3800
-Wire Wire Line
-	6050 3800 6050 3150
-Wire Wire Line
-	4950 3150 6050 3150
-Wire Wire Line
 	2300 3100 2950 3100
 Wire Wire Line
-	2650 3300 2950 3300
+	2300 3300 2950 3300
 Wire Wire Line
 	3550 3200 4700 3200
+Wire Wire Line
+	4550 6250 4800 6250
+Wire Wire Line
+	4550 6550 4800 6550
+Text HLabel 2300 3750 0    60   Input ~ 0
+MMUENA
+Wire Wire Line
+	2300 3750 4350 3750
+Connection ~ 6250 3300
+$Comp
+L 74xx:74HC14 U?
+U 3 1 5C6EA6A3
+P 4650 3450
+AR Path="/59EFC926/5C6EA6A3" Ref="U?"  Part="3"
+AR Path="/5B502B1D/5C6EA6A3" Ref="U2"  Part="3"
+F 0 "U2" H 4800 3550 50  0000 C CNN
+F 1 "74AHC14" H 4850 3350 50  0000 C CNN
+F 2 "Housings_DIP:DIP-14_W7.62mm_LongPads" H 4650 3450 50  0001 C CNN
+F 3 "" H 4650 3450 50  0001 C CNN
+	3    4650 3450
+	1    0    0    -1
+$EndComp
+Wire Wire Line
+	4950 2950 4950 3450
+Wire Wire Line
+	4350 3450 4350 3750
+Connection ~ 4350 3750
+Wire Wire Line
+	4350 3750 6250 3750
+Wire Wire Line
+	6250 3300 6250 3750
 Wire Bus Line
-	4350 1850 4350 4200
+	4350 1850 4350 2150
 $EndSCHEMATC

Commit message: Add audio output.
Parts:
- U24: symbol headquarters:74HC670 -> 74xx:74LS670
Changed lines of the file:
@@
 EESchema Schematic File Version 4
 LIBS:z80-cache
-EELAYER 26 0
+EELAYER 29 0
 EELAYER END
 $Descr USLetter 11000 8500
 encoding utf-8
-Sheet 10 10
+Sheet 10 11
 Title "Memory Management Unit"
 Date "2018-07-20"
@@
 $EndDescr
 $Comp
-L headquarters:74HC670 U24
+L 74xx:74LS670 U24
 U 1 1 5B503DBE
 P 5450 2450
-F 0 "U24" H 5150 3050 50  0000 L CNN
-F 1 "74HC670" H 5450 1850 50  0000 C CNN
+F 0 "U24" H 5150 3100 50  0000 L CNN
+F 1 "74HC670" H 5650 1700 50  0000 C CNN
 F 2 "" H 5400 2450 50  0001 C CNN
 F 3 "" H 5400 2450 50  0001 C CNN
@@
 Text HLabel 2350 1850 0    60   Input ~ 0
 D[0..3]
-Text HLabel 2300 2400 0    60   Input ~ 0
+Text HLabel 2300 2450 0    60   Input ~ 0
 WA0
-Text HLabel 2300 2500 0    60   Input ~ 0
+Text HLabel 2300 2550 0    60   Input ~ 0
 WA1
 Text HLabel 2300 3300 0    60   Input ~ 0
 ~WR
-Text HLabel 2300 2750 0    60   Input ~ 0
+Text HLabel 2300 2850 0    60   Input ~ 0
 RA0
-Text HLabel 2300 2850 0    60   Input ~ 0
+Text HLabel 2300 2950 0    60   Input ~ 0
 RA1
 Wire Wire Line
-	2300 2400 4950 2400
-Wire Wire Line
-	4950 2500 2300 2500
-Wire Wire Line
-	2300 2750 4950 2750
+	2300 2450 4950 2450
+Wire Wire Line
+	4950 2550 2300 2550
 Wire Wire Line
 	2300 2850 4950 2850
+Wire Wire Line
+	2300 2950 4950 2950
 Text HLabel 2350 1750 0    60   Output ~ 0
 A[14..17]
@@
 $EndComp
 Wire Wire Line
-	4700 3200 4700 2600
-Wire Wire Line
-	4700 2600 4950 2600
+	4700 3200 4700 2650
+Wire Wire Line
+	4700 2650 4950 2650
 $Comp
 L power:GND #PWR094
@@
 $EndComp
 Wire Wire Line
-	4950 2950 4950 3450
-Wire Wire Line
 	4350 3450 4350 3750
 Connection ~ 4350 3750
@@
 Wire Wire Line
 	6250 3300 6250 3750
+$Comp
+L power:GND #PWR0145
+U 1 1 5CBBC460
+P 5450 3350
+F 0 "#PWR0145" H 5450 3100 50  0001 C CNN
+F 1 "GND" H 5455 3177 50  0000 C CNN
+F 2 "" H 5450 3350 50  0001 C CNN
+F 3 "" H 5450 3350 50  0001 C CNN
+	1    5450 3350
+	1    0    0    -1
+$EndComp
+$Comp
+L power:VCC #PWR0144
+U 1 1 5CBBC6B8
+P 5450 1650
+F 0 "#PWR0144" H 5450 1500 50  0001 C CNN
+F 1 "VCC" H 5467 1823 50  0000 C CNN
+F 2 "" H 5450 1650 50  0001 C CNN
+F 3 "" H 5450 1650 50  0001 C CNN
+	1    5450 1650
+	1    0    0    -1
+$EndComp
+Wire Wire Line
+	4950 3050 4950 3450
 Wire Bus Line
 	4350 1850 4350 2150

Commit message: Assign footprints.
Parts:
- D2, D3, D4, D5: footprint (none) -> Diodes_SMD:D_SOT-23_ANK
- U2, U4: footprint Housings_DIP:DIP-14_W7.62mm_LongPads -> Housings_DIP:DIP-14_W7.62mm
- U24: footprint (none) -> Housings_SOIC:SOIC-16_3.9x9.9mm_Pitch1.27mm
Changed lines of the file:
@@
 F 0 "U24" H 5150 3100 50  0000 L CNN
 F 1 "74HC670" H 5650 1700 50  0000 C CNN
-F 2 "" H 5400 2450 50  0001 C CNN
+F 2 "Housings_SOIC:SOIC-16_3.9x9.9mm_Pitch1.27mm" H 5400 2450 50  0001 C CNN
 F 3 "" H 5400 2450 50  0001 C CNN
 	1    5450 2450
@@
 F 0 "D2" H 6250 3250 50  0000 C CNN
 F 1 "D_ALT" H 6250 3050 50  0000 C CNN
-F 2 "" H 6250 3150 50  0001 C CNN
+F 2 "Diodes_SMD:D_SOT-23_ANK" H 6250 3150 50  0001 C CNN
 F 3 "" H 6250 3150 50  0001 C CNN
 	1    6250 3150
@@
 F 0 "D3" H 6550 3250 50  0000 C CNN
 F 1 "D_ALT" H 6550 3050 50  0000 C CNN
-F 2 "" H 6550 3150 50  0001 C CNN
+F 2 "Diodes_SMD:D_SOT-23_ANK" H 6550 3150 50  0001 C CNN
 F 3 "" H 6550 3150 50  0001 C CNN
 	1    6550 3150
@@
 F 0 "D4" H 6850 3250 50  0000 C CNN
 F 1 "D_ALT" H 6850 3050 50  0000 C CNN
-F 2 "" H 6850 3150 50  0001 C CNN
+F 2 "Diodes_SMD:D_SOT-23_ANK" H 6850 3150 50  0001 C CNN
 F 3 "" H 6850 3150 50  0001 C CNN
 	1    6850 3150
@@
 F 0 "D5" H 7150 3250 50  0000 C CNN
 F 1 "D_ALT" H 7150 3050 50  0000 C CNN
-F 2 "" H 7150 3150 50  0001 C CNN
+F 2 "Diodes_SMD:D_SOT-23_ANK" H 7150 3150 50  0001 C CNN
 F 3 "" H 7150 3150 50  0001 C CNN
 	1    7150 3150
@@
 F 0 "U4" H 3250 3250 50  0000 C CNN
 F 1 "74AHC32" H 3250 3150 50  0000 C CNN
-F 2 "Housings_DIP:DIP-14_W7.62mm_LongPads" H 3250 3200 50  0001 C CNN
+F 2 "Housings_DIP:DIP-14_W7.62mm" H 3250 3200 50  0001 C CNN
 F 3 "" H 3250 3200 50  0001 C CNN
 	1    3250 3200
@@
 F 0 "U2" H 4800 3550 50  0000 C CNN
 F 1 "74AHC14" H 4850 3350 50  0000 C CNN
-F 2 "Housings_DIP:DIP-14_W7.62mm_LongPads" H 4650 3450 50  0001 C CNN
+F 2 "Housings_DIP:DIP-14_W7.62mm" H 4650 3450 50  0001 C CNN
 F 3 "" H 4650 3450 50  0001 C CNN
 	3    4650 3450
