File: kicad/SDcard.sch (KiCad schematic (older format))
At the start: 11 parts, among them J7 SD_Card, U25 74HCT164, U26 74AHC541, U27 74LV165, U4 74AHC32

Commit message: Add SD card footprint.
Parts:
- J7: footprint (none) -> z80_footprints:101-00405
Changed lines of the file:
@@
 EESchema Schematic File Version 4
+LIBS:zed-80-cache
 EELAYER 29 0
 EELAYER END
@@
 Sheet 9 11
 Title "SD Card Interface"
-Date "2019-04-03"
+Date "2019-04-11"
 Rev "1"
 Comp ""
@@
 F 0 "J7" H 8600 2115 50  0000 C CNN
 F 1 "SD_Card" H 8600 2024 50  0000 C CNN
-F 2 "" H 8600 1450 50  0001 C CNN
+F 2 "z80_footprints:101-00405" H 8600 1450 50  0001 C CNN
 F 3 "http://portal.fciconnect.com/Comergent//fci/drawing/10067847.pdf" H 8600 1450 50  0001 C CNN
 	1    8600 1450

Commit message: Fix schematic so that ~SDWP signal is named SDWP instead, as it is active high, not active low. There is no change to connectivity, this is only a descriptive fix.
Connections:
- net ~SDWP renamed SDWP
Changed lines of the file:
@@
 Sheet 9 11
 Title "SD Card Interface"
-Date "2019-04-15"
+Date "2019-06-02"
 Rev "1"
 Comp ""
@@
 	9900 6450 1500 6450
 Text HLabel 1500 6300 0    60   Output ~ 0
-~SDWP
+SDWP
 Text HLabel 1500 6450 0    60   Output ~ 0
 ~SDCD
