File: kicad/SIO.sch (KiCad schematic (older format))
At the start: 16 parts, among them U10 Z84C40, U11 SP232E, U12 SP232E

Commit message: Update to Kicad 5
Parts:
- C12, C13, C14, C15, C16, C17, C18, C19, C21, C22, C23: symbol C -> Device:C
- SER1, SER2: symbol DB9_Male_MountingHoles -> Connector:DB9_Male_MountingHoles
- U10: symbol Z84C40 -> headquarters:Z84C40
- U11, U12: symbol MAX232 -> Interface_UART:MAX232
Connections:
- wire segments 86 -> 91
Changed lines of the file:
@@
-EESchema Schematic File Version 2
-LIBS:power
-LIBS:device
-LIBS:transistors
-LIBS:conn
-LIBS:linear
-LIBS:regul
-LIBS:74xx
-LIBS:cmos4000
-LIBS:adc-dac
-LIBS:memory
-LIBS:xilinx
-LIBS:microcontrollers
-LIBS:dsp
-LIBS:microchip
-LIBS:analog_switches
-LIBS:motorola
-LIBS:texas
-LIBS:intel
-LIBS:audio
-LIBS:interface
-LIBS:digital-audio
-LIBS:philips
-LIBS:display
-LIBS:cypress
-LIBS:siliconi
-LIBS:opto
-LIBS:atmel
-LIBS:contrib
-LIBS:valves
-LIBS:Zilog
-LIBS:Oscillators
-LIBS:switches
-LIBS:headquarters
+EESchema Schematic File Version 4
 LIBS:z80-cache
-EELAYER 25 0
+EELAYER 26 0
 EELAYER END
 $Descr USLetter 11000 8500
@@
 $EndDescr
 $Comp
-L Z84C40 U10
+L headquarters:Z84C40 U10
 U 1 1 59D787F0
 P 4150 2900
@@
 $EndComp
 $Comp
-L GND #PWR037
+L power:GND #PWR037
 U 1 1 59D787F7
 P 4150 4500
@@
 $EndComp
 $Comp
-L VCC #PWR038
+L power:VCC #PWR038
 U 1 1 59D787FD
 P 4150 1700
@@
 NoConn ~ 4750 2500
 $Comp
-L MAX232 U11
+L Interface_UART:MAX232 U11
 U 1 1 59D7883E
 P 6450 2350
@@
 $EndComp
 $Comp
-L GND #PWR039
+L power:GND #PWR039
 U 1 1 59D78845
 P 6450 3550
@@
 $EndComp
 $Comp
-L VCC #PWR040
+L power:VCC #PWR040
 U 1 1 59D7884B
 P 6450 1150
@@
 $EndComp
 $Comp
-L GND #PWR041
+L power:GND #PWR041
 U 1 1 59D7885B
 P 4750 3000
@@
 $EndComp
 $Comp
-L GND #PWR042
+L power:GND #PWR042
 U 1 1 59D78862
 P 4750 4200
@@
 $EndComp
 $Comp
-L MAX232 U12
+L Interface_UART:MAX232 U12
 U 1 1 59D78869
 P 6450 5200
@@
 $EndComp
 $Comp
-L GND #PWR043
+L power:GND #PWR043
 U 1 1 59D78870
 P 6450 6400
@@
 $EndComp
 $Comp
-L VCC #PWR044
+L power:VCC #PWR044
 U 1 1 59D78876
 P 6450 4000
@@
 $EndComp
 $Comp
-L C C12
+L Device:C C12
 U 1 1 59D78888
 P 5650 1600
@@
 $EndComp
 $Comp
-L C C17
+L Device:C C17
 U 1 1 59D7888F
 P 7550 2400
@@
 $EndComp
 $Comp
-L C C14
+L Device:C C14
 U 1 1 59D78896
 P 7250 1600
@@
 $EndComp
 $Comp
-L GND #PWR045
+L power:GND #PWR045
 U 1 1 59D7889D
 P 7550 2550
@@
 $EndComp
 $Comp
-L C C16
+L Device:C C16
 U 1 1 59D788A4
 P 7550 1800
@@
 $EndComp
 $Comp
-L VCC #PWR046
+L power:VCC #PWR046
 U 1 1 59D788AC
 P 7550 1650
@@
 $EndComp
 $Comp
-L C C19
+L Device:C C19
 U 1 1 59D788B2
 P 7550 5250
@@
 $EndComp
 $Comp
-L C C15
+L Device:C C15
 U 1 1 59D788B9
 P 7250 4450
@@
 $EndComp
 $Comp
-L GND #PWR047
+L power:GND #PWR047
 U 1 1 59D788C0
 P 7550 5400
@@
 $EndComp
 $Comp
-L C C18
+L Device:C C18
 U 1 1 59D788C7
 P 7550 4650
@@
 $EndComp
 $Comp
-L VCC #PWR048
+L power:VCC #PWR048
 U 1 1 59D788CF
 P 7550 4500
@@
 $EndComp
 $Comp
-L C C13
+L Device:C C13
 U 1 1 59D788D5
 P 5650 4450
@@
 $EndComp
 $Comp
-L DB9_Male_MountingHoles SER1
+L Connector:DB9_Male_MountingHoles SER1
 U 1 1 59D788DC
 P 8400 2800
@@
 $EndComp
 $Comp
-L GND #PWR049
+L power:GND #PWR049
 U 1 1 59D788EF
 P 7950 2400
@@
 NoConn ~ 8100 2600
 $Comp
-L DB9_Male_MountingHoles SER2
+L Connector:DB9_Male_MountingHoles SER2
 U 1 1 59D788FA
 P 8400 5650
@@
 $EndComp
 $Comp
-L GND #PWR050
+L power:GND #PWR050
 U 1 1 59D78907
 P 7950 5250
@@
 NoConn ~ 4750 3600
 $Comp
-L GND #PWR051
+L power:GND #PWR051
 U 1 1 59D7891A
 P 8400 3400
@@
 $EndComp
 $Comp
-L GND #PWR052
+L power:GND #PWR052
 U 1 1 59D78920
 P 8400 6250
@@
 Wire Wire Line
 	3250 2700 3550 2700
-Wire Bus Line
-	3150 2100 3150 2800
 Wire Wire Line
 	5650 2850 5350 2850
@@
 B/~A
 $Comp
-L GND #PWR053
+L power:GND #PWR053
 U 1 1 59D81D49
 P 3700 7400
@@
 $EndComp
 $Comp
-L C C21
+L Device:C C21
 U 1 1 59D81D4F
 P 4250 7250
@@
 $EndComp
 $Comp
-L VCC #PWR054
+L power:VCC #PWR054
 U 1 1 59D81D56
 P 3700 7100
@@
 Connection ~ 4250 7400
 Wire Wire Line
-	3700 7400 4850 7400
-Wire Wire Line
-	3700 7100 4850 7100
-$Comp
-L C C22
+	3700 7400 4250 7400
+Wire Wire Line
+	3700 7100 4250 7100
+$Comp
+L Device:C C22
 U 1 1 59D81D90
 P 4550 7250
@@
 $EndComp
 $Comp
-L C C23
+L Device:C C23
 U 1 1 59D81D96
 P 4850 7250
@@
 	4900 2300 4750 2300
 Wire Wire Line
-	4900 1400 4900 2300
+	4900 1400 4900 2100
 Wire Wire Line
 	4900 2100 4750 2100
@@
 Wire Wire Line
 	4950 4900 2100 4900
+Wire Wire Line
+	4250 7100 4550 7100
+Wire Wire Line
+	4250 7400 4550 7400
+Wire Wire Line
+	4550 7100 4850 7100
+Wire Wire Line
+	4550 7400 4850 7400
+Wire Wire Line
+	4900 2100 4900 2300
+Wire Bus Line
+	3150 2100 3150 2800
 $EndSCHEMATC

Commit message: Assign footprints.
Parts:
- U10: footprint Housings_DIP:DIP-40_W15.24mm_Socket_LongPads -> Housings_DIP:DIP-40_W15.24mm_Socket
- U11, U12: footprint Housings_DIP:DIP-16_W7.62mm_LongPads -> Housings_DIP:DIP-16_W7.62mm
Changed lines of the file:
@@
 F 0 "U10" H 3750 3991 50  0000 L TNN
 F 1 "Z84C40" H 4550 4000 50  0000 R TNN
-F 2 "Housings_DIP:DIP-40_W15.24mm_Socket_LongPads" H 4550 4000 60  0001 C CNN
+F 2 "Housings_DIP:DIP-40_W15.24mm_Socket" H 4550 4000 60  0001 C CNN
 F 3 "" H 4550 4000 60  0001 C CNN
 	1    4150 2900
@@
 F 0 "U11" H 6350 3475 50  0000 R CNN
 F 1 "SP232E" H 6350 3400 50  0000 R CNN
-F 2 "Housings_DIP:DIP-16_W7.62mm_LongPads" H 6500 1300 50  0001 L CNN
+F 2 "Housings_DIP:DIP-16_W7.62mm" H 6500 1300 50  0001 L CNN
 F 3 "" H 6450 2450 50  0001 C CNN
 	1    6450 2350
@@
 F 0 "U12" H 6350 6325 50  0000 R CNN
 F 1 "SP232E" H 6350 6250 50  0000 R CNN
-F 2 "Housings_DIP:DIP-16_W7.62mm_LongPads" H 6500 4150 50  0001 L CNN
+F 2 "Housings_DIP:DIP-16_W7.62mm" H 6500 4150 50  0001 L CNN
 F 3 "" H 6450 5300 50  0001 C CNN
 	1    6450 5200
