File: kicad/power_reset_spares.sch (KiCad schematic (older format))
At the start: 18 parts, among them J5 USB_B, J6 PWR, SW1 KS01Q, U16 74AHC08, U2 74AHC14, U20 AP2114HA-33, U28 74HC390, U4 74AHC32, U9 74AHC02, X1 ACH20MHZ

Commit message: Assign footprints.
Parts:
- removed C24: 10uF, Capacitors_THT:CP_Radial_D5.0mm_P2.50mm, symbol Device:CP1_Small
- C30, C45: footprint (none) -> Capacitors_SMD:C_0805_HandSoldering
- C41: footprint (none) -> Capacitors_THT:C_Disc_D4.3mm_W1.9mm_P5.00mm
- R18: footprint Resistors_THT:R_Axial_DIN0204_L3.6mm_D1.6mm_P5.08mm_Horizontal -> Resistors_SMD:R_0805_HandSoldering
- U16, U2, U4, U9: footprint Housings_DIP:DIP-14_W7.62mm_LongPads -> Housings_DIP:DIP-14_W7.62mm
- U20: footprint (none) -> TO_SOT_Packages_SMD:SOT-223-3_TabPin2
- U28: footprint (none) -> Housings_SSOP:TSSOP-16_4.4x5mm_Pitch0.65mm
Changed lines of the file:
@@
 F 0 "U16" H 1100 1000 50  0000 C CNN
 F 1 "74AHC08" H 1100 900 50  0000 C CNN
-F 2 "Housings_DIP:DIP-14_W7.62mm_LongPads" H 1100 950 50  0001 C CNN
+F 2 "Housings_DIP:DIP-14_W7.62mm" H 1100 950 50  0001 C CNN
 F 3 "" H 1100 950 50  0001 C CNN
 	2    1100 950
@@
 F 0 "U16" H 1100 1450 50  0000 C CNN
 F 1 "74AHC08" H 1100 1350 50  0000 C CNN
-F 2 "Housings_DIP:DIP-14_W7.62mm_LongPads" H 1100 1400 50  0001 C CNN
+F 2 "Housings_DIP:DIP-14_W7.62mm" H 1100 1400 50  0001 C CNN
 F 3 "" H 1100 1400 50  0001 C CNN
 	3    1100 1400
@@
 F 0 "U16" H 1100 1950 50  0000 C CNN
 F 1 "74AHC08" H 1100 1850 50  0000 C CNN
-F 2 "Housings_DIP:DIP-14_W7.62mm_LongPads" H 1100 1900 50  0001 C CNN
+F 2 "Housings_DIP:DIP-14_W7.62mm" H 1100 1900 50  0001 C CNN
 F 3 "" H 1100 1900 50  0001 C CNN
 	4    1100 1900
@@
 F 0 "U9" H 1900 1000 50  0000 C CNN
 F 1 "74AHC02" H 1950 900 50  0000 C CNN
-F 2 "Housings_DIP:DIP-14_W7.62mm_LongPads" H 1900 950 50  0001 C CNN
+F 2 "Housings_DIP:DIP-14_W7.62mm" H 1900 950 50  0001 C CNN
 F 3 "" H 1900 950 50  0001 C CNN
 	4    1900 950
@@
 F 0 "R18" V 6630 1400 50  0000 C CNN
 F 1 "10K" V 6550 1400 50  0000 C CNN
-F 2 "Resistors_THT:R_Axial_DIN0204_L3.6mm_D1.6mm_P5.08mm_Horizontal" V 6480 1400 50  0001 C CNN
+F 2 "Resistors_SMD:R_0805_HandSoldering" V 6480 1400 50  0001 C CNN
 F 3 "" H 6550 1400 50  0001 C CNN
 	1    6550 1400
@@
 $EndComp
 $Comp
-L Device:CP1_Small C?
-U 1 1 5CB1CFB6
-P 6850 1250
-AR Path="/5CB1CFB6" Ref="C?"  Part="1"
-AR Path="/59EFC926/5CB1CFB6" Ref="C24"  Part="1"
-F 0 "C24" H 6860 1320 50  0000 L CNN
-F 1 "10uF" H 6860 1170 50  0000 L CNN
-F 2 "Capacitors_THT:CP_Radial_D5.0mm_P2.50mm" H 6850 1250 50  0001 C CNN
-F 3 "" H 6850 1250 50  0001 C CNN
-	1    6850 1250
-	1    0    0    -1
-$EndComp
-$Comp
 L Connector:USB_B J?
 U 1 1 5CB1CFBD
@@
 F 0 "C30" H 8975 1300 50  0000 L CNN
 F 1 "4.7uF" H 8975 1100 50  0000 L CNN
-F 2 "" H 8988 1050 50  0001 C CNN
+F 2 "Capacitors_SMD:C_0805_HandSoldering" H 8988 1050 50  0001 C CNN
 F 3 "" H 8950 1200 50  0001 C CNN
 	1    8950 1200
@@
 Connection ~ 6550 950
 Wire Wire Line
-	6850 1150 6850 950
-Connection ~ 6850 950
-Wire Wire Line
-	6850 1550 6850 1350
-Connection ~ 6850 1550
-Wire Wire Line
 	7100 1550 7100 1300
 Connection ~ 7100 950
@@
 Wire Wire Line
 	6000 1550 6550 1550
-Wire Wire Line
-	6550 1550 6850 1550
-Wire Wire Line
-	6550 950  6850 950
-Wire Wire Line
-	6850 950  7100 950
-Wire Wire Line
-	6850 1550 7100 1550
 Wire Wire Line
 	8750 950  8950 950
@@
 F 0 "U2" H 7050 2950 50  0000 C CNN
 F 1 "74AHC14" H 7100 2750 50  0000 C CNN
-F 2 "Housings_DIP:DIP-14_W7.62mm_LongPads" H 6900 2850 50  0001 C CNN
+F 2 "Housings_DIP:DIP-14_W7.62mm" H 6900 2850 50  0001 C CNN
 F 3 "http://www.ti.com/lit/ds/symlink/sn74ahc14.pdf" H 6900 2850 50  0001 C CNN
 	1    6900 2850
@@
 F 0 "U2" H 8050 2950 50  0000 C CNN
 F 1 "74AHC14" H 8100 2750 50  0000 C CNN
-F 2 "Housings_DIP:DIP-14_W7.62mm_LongPads" H 7900 2850 50  0001 C CNN
+F 2 "Housings_DIP:DIP-14_W7.62mm" H 7900 2850 50  0001 C CNN
 F 3 "" H 7900 2850 50  0001 C CNN
 	2    7900 2850
@@
 F 0 "U4" H 3750 1000 50  0000 C CNN
 F 1 "74AHC32" H 3750 900 50  0000 C CNN
-F 2 "Housings_DIP:DIP-14_W7.62mm_LongPads" H 3750 950 50  0001 C CNN
+F 2 "Housings_DIP:DIP-14_W7.62mm" H 3750 950 50  0001 C CNN
 F 3 "" H 3750 950 50  0001 C CNN
 	4    3750 950
@@
 F 0 "U2" H 2950 1050 50  0000 C CNN
 F 1 "74AHC14" H 3000 850 50  0000 C CNN
-F 2 "Housings_DIP:DIP-14_W7.62mm_LongPads" H 2800 950 50  0001 C CNN
+F 2 "Housings_DIP:DIP-14_W7.62mm" H 2800 950 50  0001 C CNN
 F 3 "" H 2800 950 50  0001 C CNN
 	4    2800 950
@@
 F 0 "U28" H 7500 4200 50  0000 C CNN
 F 1 "74HC390" H 7500 3600 50  0000 C CNN
-F 2 "" H 7500 3950 50  0001 C CNN
+F 2 "Housings_SSOP:TSSOP-16_4.4x5mm_Pitch0.65mm" H 7500 3950 50  0001 C CNN
 F 3 "http://www.ti.com/lit/gpn/sn74LS390" H 7500 3950 50  0001 C CNN
 	1    7500 3950
@@
 F 0 "U28" H 7500 5150 50  0000 C CNN
 F 1 "74HC390" H 7500 4550 50  0000 C CNN
-F 2 "" H 7500 4900 50  0001 C CNN
+F 2 "Housings_SSOP:TSSOP-16_4.4x5mm_Pitch0.65mm" H 7500 4900 50  0001 C CNN
 F 3 "http://www.ti.com/lit/gpn/sn74LS390" H 7500 4900 50  0001 C CNN
 	2    7500 4900
@@
 F 0 "U28" H 6100 6150 50  0000 L CNN
 F 1 "74HC390" H 6100 5450 50  0000 L CNN
-F 2 "" H 6050 5800 50  0001 C CNN
+F 2 "Housings_SSOP:TSSOP-16_4.4x5mm_Pitch0.65mm" H 6050 5800 50  0001 C CNN
 F 3 "http://www.ti.com/lit/gpn/sn74LS390" H 6050 5800 50  0001 C CNN
 	3    6050 5800
@@
 F 0 "C41" H 5600 5850 50  0000 L CNN
 F 1 "0.1uF" H 5600 5650 50  0000 L CNN
-F 2 "" H 5588 5600 50  0001 C CNN
+F 2 "Capacitors_THT:C_Disc_D4.3mm_W1.9mm_P5.00mm" H 5588 5600 50  0001 C CNN
 F 3 "~" H 5550 5750 50  0001 C CNN
 	1    5550 5750
@@
 F 0 "U20" H 8000 1100 50  0000 C CNN
 F 1 "AP2114HA-33" H 8450 700 50  0000 C CNN
-F 2 "" H 8150 1175 50  0001 C CIN
+F 2 "TO_SOT_Packages_SMD:SOT-223-3_TabPin2" H 8150 1175 50  0001 C CIN
 F 3 "" H 8150 900 50  0001 C CNN
 	1    8150 950
@@
 F 0 "C45" H 7675 1300 50  0000 L CNN
 F 1 "4.7uF" H 7675 1100 50  0000 L CNN
-F 2 "" H 7688 1050 50  0001 C CNN
+F 2 "Capacitors_SMD:C_0805_HandSoldering" H 7688 1050 50  0001 C CNN
 F 3 "" H 7650 1200 50  0001 C CNN
 	1    7650 1200
@@
 Wire Wire Line
 	7650 950  7850 950
+Wire Wire Line
+	6550 1550 7100 1550
+Wire Wire Line
+	6550 950  7100 950
 $EndSCHEMATC

Commit message: First pass layout of revised board complete.
Parts:
- added C20, C26, C3, C5: 0.1uF, Capacitors_THT:C_Disc_D4.3mm_W1.9mm_P5.00mm, symbol Device:C
- added H1, H2, H3, H4: 3.2mm M3, Mounting_Holes:MountingHole_3.2mm_M3_Pad, symbol Mechanical:MountingHole_Pad
- added unit 5 of U16
- added unit 7 of U2
- added unit 5 of U4
- added unit 5 of U9
Connections:
- net GND: now also C20.2, C26.2, C3.2, C5.2, H1.1, H2.1, H3.1, H4.1, U16.7 (GND), U2.7 (GND), U4.7 (GND), U9.7 (GND)
- net VCC: now also C20.1, C26.1, C3.1, C5.1, U16.14 (VCC), U2.14 (VCC), U4.14 (VCC), U9.14 (VCC)
Other:
- note added: "Clocks"
- note added: "Mounting holes"
- note added: "Power"
- note added: "Power units & decoupling"
- note added: "Reset"
- note added: "Spares"
- note removed: "Near\nU28"
- moved on the sheet: C1, C30, C41, C45, D1, J5, J6, R1, R18, SW1, U16B, U16C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
